File: KiCAD files/TVZ_KTM_ApplicationBoard.kicad_sch (KiCad schematic)
At the start: 65 parts, among them J1 Conn_02x19_Odd_Even, J2 Conn_02x19_Odd_Even, J3 Conn_02x19_Odd_Even, J4 Conn_02x19_Odd_Even, SW1 EG1271A, SW2 EG1271A, SW3 EG1271A, SW4 EG1271A, U1 LM75B, U2 MCP2551-I-P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

Commit message: update
Connections:
- net +3V3: no longer J3.16 (Pin_16)
- net GND: now also J2.32 (Pin_32), J4.32 (Pin_32)
- no-connect marks 91 -> 90
Changed lines of the file:
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@@
   (no_connect (at 210.82 63.5))
   (no_connect (at 261.62 30.48))
+  (no_connect (at 223.52 45.72))
   (no_connect (at 223.52 38.1))
   (no_connect (at 29.21 62.865))
@@
   (no_connect (at 261.62 68.58))
   (no_connect (at 80.01 70.485))
-  (no_connect (at 80.01 62.865))
   (no_connect (at 41.91 60.325))
   (no_connect (at 29.21 42.545))
@@
   (no_connect (at 210.82 58.42))
   (no_connect (at 210.82 43.18))
-  (no_connect (at 223.52 45.72))
   (no_connect (at 80.01 29.845))
   (no_connect (at 223.52 68.58))
@@
   (no_connect (at 80.01 65.405))
   (no_connect (at 248.92 68.58))
-  (no_connect (at 261.62 63.5))
+  (no_connect (at 223.52 43.18))
   (no_connect (at 223.52 60.96))
   (no_connect (at 223.52 55.88))
@@
     (stroke (width 0) (type default))
   )
-  (wire (pts (xy 231.775 43.18) (xy 231.775 41.275))
-    (stroke (width 0) (type default))
-  )
   (wire (pts (xy 179.07 89.535) (xy 179.07 90.805))
     (stroke (width 0) (type default))
@@
     (stroke (width 0) (type default))
   )
-  (wire (pts (xy 223.52 43.18) (xy 231.775 43.18))
-    (stroke (width 0) (type default))
-  )
   (wire (pts (xy 41.91 32.385) (xy 45.72 32.385))
     (stroke (width 0) (type default))
@@
     (stroke (width 0) (type default))
   )
+  (wire (pts (xy 80.01 62.865) (xy 85.725 62.865))
+    (stroke (width 0) (type default))
+  )
   (wire (pts (xy 150.495 96.52) (xy 154.94 96.52))
     (stroke (width 0) (type default))
@@
     (stroke (width 0) (type default))
   )
+  (wire (pts (xy 267.335 63.5) (xy 261.62 63.5))
+    (stroke (width 0) (type default))
+  )
   (wire (pts (xy 51.435 86.995) (xy 51.435 88.9))
     (stroke (width 0) (type default))
@@
     (stroke (width 0) (type default))
   )
+  (wire (pts (xy 267.335 66.04) (xy 267.335 63.5))
+    (stroke (width 0) (type default))
+  )
   (wire (pts (xy 131.445 145.415) (xy 133.985 145.415))
     (stroke (width 0) (type default))
@@
     (stroke (width 0) (type default))
   )
+  (wire (pts (xy 85.725 66.675) (xy 85.725 62.865))
+    (stroke (width 0) (type default))
+  )
   (wire (pts (xy 42.545 100.33) (xy 42.545 99.695))
     (stroke (width 0) (type default))
@@
     )
   )
-  (symbol (lib_id "power:+3V3") (at 231.775 41.275 0) (unit 1)
+  (symbol (lib_name "GND_18") (lib_id "power:GND") (at 85.725 66.675 0) (unit 1)
     (in_bom yes) (on_board yes) (dnp no) (fields_autoplaced)
-    (property "Reference" "#PWR026" (at 231.775 45.085 0)
+    (property "Reference" "#PWR039" (at 85.725 73.025 0)
       (effects (font (size 1.27 1.27)) hide)
     )
-    (property "Value" "+3V3" (at 231.775 37.6992 0)
+    (property "Value" "GND" (at 85.725 71.1184 0)
       (effects (font (size 1.27 1.27)))
     )
-    (property "Footprint" "" (at 231.775 41.275 0)
+    (property "Footprint" "" (at 85.725 66.675 0)
       (effects (font (size 1.27 1.27)) hide)
     )
-    (property "Datasheet" "" (at 231.775 41.275 0)
+    (property "Datasheet" "" (at 85.725 66.675 0)
       (effects (font (size 1.27 1.27)) hide)
     )
@@
       (project "TVZ_KTM_ApplicationBoard"
         (path "/e6e1ba2c-0a46-4bca-b3ad-33e778ea698b"
-          (reference "#PWR026") (unit 1)
+          (reference "#PWR039") (unit 1)
         )
       )
@@
     )
   )
+  (symbol (lib_name "GND_8") (lib_id "power:GND") (at 267.335 66.04 0) (unit 1)
+    (in_bom yes) (on_board yes) (dnp no) (fields_autoplaced)
+    (property "Reference" "#PWR024" (at 267.335 72.39 0)
+      (effects (font (size 1.27 1.27)) hide)
+    )
+    (property "Value" "GND" (at 267.335 70.4834 0)
+      (effects (font (size 1.27 1.27)))
+    )
+    (property "Footprint" "" (at 267.335 66.04 0)
+      (effects (font (size 1.27 1.27)) hide)
+    )
+    (property "Datasheet" "" (at 267.335 66.04 0)
+      (effects (font (size 1.27 1.27)) hide)
+    )
+    (pin "1")
+    (instances
+      (project "TVZ_KTM_ApplicationBoard"
+        (path "/e6e1ba2c-0a46-4bca-b3ad-33e778ea698b"
+          (reference "#PWR024") (unit 1)
+        )
+      )
+    )
+  )
   (symbol (lib_id "Interface_CAN_LIN:MCP2551-I-P") (at 179.07 100.965 0) (mirror y) (unit 1)
     (in_bom yes) (on_board yes) (dnp no)
@@
     )
   )
-  (symbol (lib_id "power:+5V") (at 179.07 88.265 0) (unit 1)
-    (in_bom yes) (on_board yes) (dnp no) (fields_autoplaced)
-    (property "Reference" "#PWR0105" (at 179.07 92.075 0)
-      (effects (font (size 1.27 1.27)) hide)
-    )
-    (property "Value" "+5V" (at 179.07 84.6892 0)
-      (effects (font (size 1.27 1.27)))
-    )
-    (property "Footprint" "" (at 179.07 88.265 0)
-      (effects (font (size 1.27 1.27)) hide)
-    )
-    (property "Datasheet" "" (at 179.07 88.265 0)
-      (effects (font (size 1.27 1.27)) hide)
-    )
-    (pin "1")
-    (instances
-      (project "TVZ_KTM_ApplicationBoard"
-        (path "/e6e1ba2c-0a46-4bca-b3ad-33e778ea698b"
-          (reference "#PWR0105") (unit 1)
-        )
-      )
-    )
-  )
   (symbol (lib_id "Connector:TestPoint") (at 185.42 55.245 0) (unit 1)
     (in_bom yes) (on_board yes) (dnp no) (fields_autoplaced)
@@
         )
       )
+    )
+  )
+  (symbol (lib_id "power:+5V") (at 179.07 88.265 0) (unit 1)
+    (in_bom yes) (on_board yes) (dnp no) (fields_autoplaced)
+    (property "Reference" "#PWR026" (at 179.07 92.075 0)
+      (effects (font (size 1.27 1.27)) hide)
+    )
+    (property "Value" "+5V" (at 179.07 84.6892 0)
+      (effects (font (size 1.27 1.27)))
+    )
+    (property "Footprint" "" (at 179.07 88.265 0)
+      (effects (font (size 1.27 1.27)) hide)
+    )
+    (property "Datasheet" "" (at 179.07 88.265 0)
+      (effects (font (size 1.27 1.27)) hide)
+    )
+    (pin "1")
+    (instances
+      (project "TVZ_KTM_ApplicationBoard"
+        (path "/e6e1ba2c-0a46-4bca-b3ad-33e778ea698b"
+          (reference "#PWR026") (unit 1)
+        )
+      )

Commit message: update
Parts:
- added U4, U6: ~, symbol Symbol:NucleoF446RE-1
- added U5, U7: ~, symbol Symbol:NucleoF446RE-2
Other:
- note added: "- obratiti pozornost na MSB i LSB kod rasporeda sklopki, LEDica i ostalih elemenata"

Commit message: update
Parts:
- removed D1, D2, D3, D4: BLUE, LED_SMD:LED_1206_3216Metric, symbol Device:LED_Small
- removed D10, D11, D12, D9: RED, LED_SMD:LED_1206_3216Metric, symbol Device:LED_Small
- removed D13: boja, LED_SMD:LED_1206_3216Metric, symbol Device:LED_Small
- removed D5, D6, D7, D8: GREEN, LED_SMD:LED_1206_3216Metric, symbol Device:LED_Small
- removed J1, J2, J3, J4: Conn_02x19_Odd_Even, Connector_PinSocket_2.54mm:PinSocket_2x19_P2.54mm_Vertical, symbol Connector_Generic:Conn_02x19_Odd_Even
- removed JP4, JP5: Jumper_3_Open, Connector_PinHeader_2.54mm:PinHeader_1x03_P2.54mm_Vertical, symbol Jumper:Jumper_3_Open
- removed R10, R11, R12, R13, R14, R15, R16, R17, R20, R6, R7, R8, R9: 220, Resistor_SMD:R_0805_2012Metric, symbol Device:R_Small
- removed SW1, SW2, SW3, SW4: EG1271A, Footprint:EG1271A, symbol Switch:SW_SPDT
- removed TP12, TP13, TP2: TestPoint, Footprint:KEYS4952, symbol Connector:TestPoint
- removed U4, U6: ~, symbol Symbol:NucleoF446RE-1
- removed U5, U7: ~, symbol Symbol:NucleoF446RE-2
- added JP2, JP3: Jumper_3_Open, Connector_PinHeader_2.54mm:PinHeader_1x03_P2.54mm_Vertical, symbol Jumper:Jumper_3_Open
Connections:
- net +3V3: now also JP2.1 (A), JP3.1 (A)
- net GND: now also JP2.3 (B), JP3.3 (B)
- net at R4.2: now also JP2.2 (C)
- net at R5.2: now also JP3.2 (C)
- net PA10_1 renamed USART_TX(M) >> USART_RX(S)
- net PA11_1 renamed CAN_RD(M)
- net PA11_2 renamed CAN_RD(S)
- net PA12_1 renamed CAN_TD(M)
- net PA12_2 renamed CAN_TD(S)
- net PA9_1 renamed USART_RX(M) >> USART_TX(S)
- net PB8_1 renamed I2C_SCL
- net I2C_SCL: now also TP5.1; no longer TP6.1
- net PB9_1 renamed I2C_SDA
- net I2C_SDA: now also TP6.1; no longer TP5.1
- no-connect marks 90 -> 3
Other:
- added sheet Master (Master.kicad_sch)
- added sheet Slave (Slave.kicad_sch)
- note removed: "DAC MASTER"
- note removed: "MASTER"
- note removed: "RX MASTER"
- note removed: "SLAVE"
- note removed: "TX MASTER"
- note removed: "na desnu stranu plave"
- note removed: "na lijevu stranu idu crvene i zelene"
- note removed: "sklopke idu na lijevu stranu"
- moved on the sheet: C2, C3, R18, R19, TP10, TP11, TP14, U2, U3

Commit message: update
Connections:
- net USART_RX(M) >> USART_TX(S): now also TP7.1; no longer TP8.1
- net USART_TX(M) >> USART_RX(S): now also TP8.1; no longer TP7.1
- net PA4_2: no longer names the net of TP14.1
- net PA7_BUSY renamed BUSY
- net PA8_STROBE renamed STROBE
- no-connect marks 3 -> 4
Other:
- note added: "TODO: - obratiti pozornost na MSB i LSB kod rasporeda sklopki, LEDica i ostalih elemenata - provjeriti TP14 (jel treba DAC slave?) - MCP2551 naponsko djelilo ( RX na 3.3V?) - LED13 nije spojena, čemu ono služi? (mislim da je za DAC slave?) - sitotisak pinovi"
- note removed: "- obratiti pozornost na MSB i LSB kod rasporeda sklopki, LEDica i ostalih elemenata"
- moved on the sheet: TP10, TP11, TP14, TP7, TP8
Changed lines of the file:
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@@
   )
   (no_connect (at 181.61 119.38))
+  (no_connect (at 150.495 160.02))
   (no_connect (at 73.025 113.03))
   (no_connect (at 254.635 119.38))
@@
     (stroke (width 0) (type default))
   )
-  (polyline (pts (xy 440.055 186.69) (xy 504.19 186.69))
-    (stroke (width 0) (type default))
-  )
   (wire (pts (xy 194.31 104.14) (xy 194.31 105.41))
     (stroke (width 0) (type default))
@@
   )
   (wire (pts (xy 229.235 119.38) (xy 227.33 119.38))
-    (stroke (width 0) (type default))
-  )
-  (polyline (pts (xy 339.725 186.69) (xy 439.42 186.69))
     (stroke (width 0) (type default))
   )
@@
     (effects (font (size 2.54 2.54) (thickness 0.508) bold) (justify left bottom))
   )
-  (text "- obratiti pozornost na MSB i LSB kod rasporeda sklopki, LEDica i ostalih elemenata"
+  (text "TODO:\n- obratiti pozornost na MSB i LSB kod rasporeda sklopki, LEDica i ostalih elemenata\n- provjeriti TP14 (jel treba DAC slave?)\n- MCP2551 naponsko djelilo ( RX na 3.3V?)\n- LED13 nije spojena, čemu ono služi? (mislim da je za DAC slave?)\n- sitotisak pinovi"
     (at 15.875 191.77 0)
     (effects (font (size 1.27 1.27)) (justify left bottom))
   )
-  (text "DAC SLAVE" (at 202.565 -7.62 0)
+  (text "DAC SLAVE" (at 147.955 174.625 0)
     (effects (font (size 1.27 1.27)) (justify left bottom))
   )
-  (text "BUSY" (at 162.56 -6.985 0)
+  (text "BUSY" (at 107.95 175.26 0)
     (effects (font (size 1.27 1.27)) (justify left bottom))
   )
@@
     )
   )
-  (global_label "PA4_2" (shape input) (at 205.105 -22.225 270) (fields_autoplaced)
-    (effects (font (size 1.27 1.27)) (justify right))
-    (property "Intersheetrefs" "${INTERSHEET_REFS}" (at 205.1844 -14.0667 90)
-      (effects (font (size 1.27 1.27)) (justify right) hide)
-    )
-  )
   (global_label "CAN_RD(S)" (shape input) (at 254.635 114.3 0) (fields_autoplaced)
     (effects (font (size 1.27 1.27)) (justify left))
@@
     )
   )
-  (global_label "PA8_STROBE" (shape input) (at 125.73 -51.435 270) (fields_autoplaced)
+  (global_label "STROBE" (shape input) (at 99.06 158.75 270) (fields_autoplaced)
     (effects (font (size 1.27 1.27)) (justify right))
-    (property "Intersheetrefs" "${INTERSHEET_REFS}" (at 125.6506 -37.2895 90)
+    (property "Intersheetrefs" "${INTERSHEET_REFS}" (at 99.06 168.9318 90)
       (effects (font (size 1.27 1.27)) (justify right) hide)
     )
   )
-  (global_label "PA7_BUSY" (shape input) (at 165.735 -23.495 270) (fields_autoplaced)
+  (global_label "BUSY" (shape input) (at 111.125 158.75 270) (fields_autoplaced)
     (effects (font (size 1.27 1.27)) (justify right))
-    (property "Intersheetrefs" "${INTERSHEET_REFS}" (at 165.6556 -11.6476 90)
+    (property "Intersheetrefs" "${INTERSHEET_REFS}" (at 111.125 166.6338 90)
       (effects (font (size 1.27 1.27)) (justify right) hide)
     )
@@
     )
   )
-  (symbol (lib_id "Connector:TestPoint") (at 165.735 -23.495 0) (unit 1)
-    (in_bom yes) (on_board yes) (dnp no) (fields_autoplaced)
-    (property "Reference" "TP10" (at 167.132 -26.3632 0)
-      (effects (font (size 1.27 1.27)) (justify left))
-    )
-    (property "Value" "TestPoint" (at 167.132 -25.0948 0)
-      (effects (font (size 1.27 1.27)) (justify left) hide)
-    )
-    (property "Footprint" "Footprint:KEYS4952" (at 170.815 -23.495 0)
-      (effects (font (size 1.27 1.27)) hide)
-    )
-    (property "Datasheet" "~" (at 170.815 -23.495 0)
+  (symbol (lib_id "Connector:TestPoint") (at 111.125 158.75 0) (unit 1)
+    (in_bom yes) (on_board yes) (dnp no) (fields_autoplaced)
+    (property "Reference" "TP10" (at 112.522 155.8818 0)
+      (effects (font (size 1.27 1.27)) (justify left))
+    )
+    (property "Value" "TestPoint" (at 112.522 157.1502 0)
+      (effects (font (size 1.27 1.27)) (justify left) hide)
+    )
+    (property "Footprint" "Footprint:KEYS4952" (at 116.205 158.75 0)
+      (effects (font (size 1.27 1.27)) hide)
+    )
+    (property "Datasheet" "~" (at 116.205 158.75 0)
       (effects (font (size 1.27 1.27)) hide)
     )
@@
     )
   )
-  (symbol (lib_id "Connector:TestPoint") (at 226.06 41.275 0) (unit 1)
-    (in_bom yes) (on_board yes) (dnp no) (fields_autoplaced)
-    (property "Reference" "TP7" (at 227.457 38.4068 0)
-      (effects (font (size 1.27 1.27)) (justify left))
-    )
-    (property "Value" "TestPoint" (at 227.457 39.6752 0)
-      (effects (font (size 1.27 1.27)) (justify left) hide)
-    )
-    (property "Footprint" "Footprint:KEYS4952" (at 231.14 41.275 0)
-      (effects (font (size 1.27 1.27)) hide)
-    )
-    (property "Datasheet" "~" (at 231.14 41.275 0)
+  (symbol (lib_id "Connector:TestPoint") (at 238.76 41.275 0) (unit 1)
+    (in_bom yes) (on_board yes) (dnp no) (fields_autoplaced)
+    (property "Reference" "TP7" (at 240.157 38.4068 0)
+      (effects (font (size 1.27 1.27)) (justify left))
+    )
+    (property "Value" "TestPoint" (at 240.157 39.6752 0)
+      (effects (font (size 1.27 1.27)) (justify left) hide)
+    )
+    (property "Footprint" "Footprint:KEYS4952" (at 243.84 41.275 0)
+      (effects (font (size 1.27 1.27)) hide)
+    )
+    (property "Datasheet" "~" (at 243.84 41.275 0)
       (effects (font (size 1.27 1.27)) hide)
     )
@@
     )
   )
-  (symbol (lib_id "Connector:TestPoint") (at 205.105 -22.225 0) (unit 1)
-    (in_bom yes) (on_board yes) (dnp no) (fields_autoplaced)
-    (property "Reference" "TP14" (at 206.502 -25.0932 0)
-      (effects (font (size 1.27 1.27)) (justify left))
-    )
-    (property "Value" "TestPoint" (at 206.502 -23.8248 0)
-      (effects (font (size 1.27 1.27)) (justify left) hide)
-    )
-    (property "Footprint" "Footprint:KEYS4952" (at 210.185 -22.225 0)
-      (effects (font (size 1.27 1.27)) hide)
-    )
-    (property "Datasheet" "~" (at 210.185 -22.225 0)
+  (symbol (lib_id "Connector:TestPoint") (at 150.495 160.02 0) (unit 1)
+    (in_bom yes) (on_board yes) (dnp no) (fields_autoplaced)
+    (property "Reference" "TP14" (at 151.892 157.1518 0)
+      (effects (font (size 1.27 1.27)) (justify left))
+    )
+    (property "Value" "TestPoint" (at 151.892 158.4202 0)
+      (effects (font (size 1.27 1.27)) (justify left) hide)
+    )
+    (property "Footprint" "Footprint:KEYS4952" (at 155.575 160.02 0)
+      (effects (font (size 1.27 1.27)) hide)
+    )
+    (property "Datasheet" "~" (at 155.575 160.02 0)
       (effects (font (size 1.27 1.27)) hide)
     )
@@
     )
   )
-  (symbol (lib_id "Connector:TestPoint") (at 125.73 -51.435 0) (unit 1)
-    (in_bom yes) (on_board yes) (dnp no) (fields_autoplaced)
-    (property "Reference" "TP11" (at 127.127 -54.3032 0)
-      (effects (font (size 1.27 1.27)) (justify left))
-    )
-    (property "Value" "TestPoint" (at 127.127 -53.0348 0)
-      (effects (font (size 1.27 1.27)) (justify left) hide)
-    )
-    (property "Footprint" "Footprint:KEYS4952" (at 130.81 -51.435 0)
-      (effects (font (size 1.27 1.27)) hide)
-    )
-    (property "Datasheet" "~" (at 130.81 -51.435 0)
+  (symbol (lib_id "Connector:TestPoint") (at 99.06 158.75 0) (unit 1)
+    (in_bom yes) (on_board yes) (dnp no) (fields_autoplaced)
+    (property "Reference" "TP11" (at 100.457 155.8818 0)
+      (effects (font (size 1.27 1.27)) (justify left))
+    )
+    (property "Value" "TestPoint" (at 100.457 157.1502 0)
+      (effects (font (size 1.27 1.27)) (justify left) hide)
+    )
+    (property "Footprint" "Footprint:KEYS4952" (at 104.14 158.75 0)
+      (effects (font (size 1.27 1.27)) hide)
+    )
+    (property "Datasheet" "~" (at 104.14 158.75 0)
       (effects (font (size 1.27 1.27)) hide)
     )
@@
     )
   )
-  (symbol (lib_id "Connector:TestPoint") (at 238.76 41.275 0) (unit 1)
-    (in_bom yes) (on_board yes) (dnp no) (fields_autoplaced)
-    (property "Reference" "TP8" (at 240.157 38.4068 0)
-      (effects (font (size 1.27 1.27)) (justify left))
-    )
-    (property "Value" "TestPoint" (at 240.157 39.6752 0)
-      (effects (font (size 1.27 1.27)) (justify left) hide)
-    )
-    (property "Footprint" "Footprint:KEYS4952" (at 243.84 41.275 0)
-      (effects (font (size 1.27 1.27)) hide)
-    )
-    (property "Datasheet" "~" (at 243.84 41.275 0)
-      (effects (font (size 1.27 1.27)) hide)
-    )
+  (symbol (lib_id "Connector:TestPoint") (at 226.06 41.275 0) (unit 1)
+    (in_bom yes) (on_board yes) (dnp no) (fields_autoplaced)
+    (property "Reference" "TP8" (at 227.457 38.4068 0)
+      (effects (font (size 1.27 1.27)) (justify left))
+    )
+    (property "Value" "TestPoint" (at 227.457 39.6752 0)
+      (effects (font (size 1.27 1.27)) (justify left) hide)
+    )
+    (property "Footprint" "Footprint:KEYS4952" (at 231.14 41.275 0)
+      (effects (font (size 1.27 1.27)) hide)
+    )
+    (property "Datasheet" "~" (at 231.14 41.275 0)
+      (effects (font (size 1.27 1.27)) hide)
+    )
