File: KiCAD files/TVZ_KTM_ApplicationBoard.kicad_sch (KiCad schematic)
At the start: 28 parts, among them U1 LM75B, U2 MCP2551-I-P, U3 MCP2551-I-P

Commit message: update
Connections:
- net I2C_SCL: now also TP6.1; no longer TP5.1
- net I2C_SDA: now also TP5.1; no longer TP6.1
Changed lines of the file:
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@@
     )
   )
-  (global_label "I2C_SCL" (shape input) (at 57.785 130.175 270) (fields_autoplaced)
-    (effects (font (size 1.27 1.27)) (justify right))
-    (property "Intersheetrefs" "${INTERSHEET_REFS}" (at 57.785 140.7197 90)
+  (global_label "I2C_SCL" (shape input) (at 53.975 130.175 270) (fields_autoplaced)
+    (effects (font (size 1.27 1.27)) (justify right))
+    (property "Intersheetrefs" "${INTERSHEET_REFS}" (at 53.975 140.7197 90)
       (effects (font (size 1.27 1.27)) (justify right) hide)
     )
@@
     )
   )
-  (global_label "I2C_SDA" (shape input) (at 53.975 130.175 270) (fields_autoplaced)
-    (effects (font (size 1.27 1.27)) (justify right))
-    (property "Intersheetrefs" "${INTERSHEET_REFS}" (at 53.975 140.7802 90)
+  (global_label "I2C_SDA" (shape input) (at 57.785 130.175 270) (fields_autoplaced)
+    (effects (font (size 1.27 1.27)) (justify right))
+    (property "Intersheetrefs" "${INTERSHEET_REFS}" (at 57.785 140.7802 90)
       (effects (font (size 1.27 1.27)) (justify right) hide)
     )
@@
   )
   (symbol (lib_id "Jumper:Jumper_3_Open") (at 115.57 94.615 270) (unit 1)
-    (in_bom yes) (on_board yes) (dnp no) (fields_autoplaced)
+    (in_bom yes) (on_board yes) (dnp no)
     (property "Reference" "JP1" (at 117.7042 95.0488 90)
       (effects (font (size 1.27 1.27)) (justify left))

Commit message: update
Connections:
- net GND: now also TP14.1
- no-connect marks 4 -> 3
Other:
- note removed: "DAC SLAVE"
Changed lines of the file:
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@@
   )
   (no_connect (at 181.61 119.38))
-  (no_connect (at 150.495 160.02))
   (no_connect (at 73.025 113.03))
   (no_connect (at 254.635 119.38))
@@
   (text "TODO:\n- obratiti pozornost na MSB i LSB kod rasporeda sklopki, LEDica i ostalih elemenata\n- provjeriti TP14 (jel treba DAC slave?)\n- MCP2551 naponsko djelilo ( RX na 3.3V?)\n- LED13 nije spojena, čemu ono služi? (mislim da je za DAC slave?)\n- sitotisak pinovi"
     (at 15.875 191.77 0)
-    (effects (font (size 1.27 1.27)) (justify left bottom))
-  )
-  (text "DAC SLAVE" (at 147.955 174.625 0)
     (effects (font (size 1.27 1.27)) (justify left bottom))
   )
@@
         )
       )
+    )
+  )
+  (symbol (lib_name "GND_29") (lib_id "power:GND") (at 150.495 160.02 0) (unit 1)
+    (in_bom yes) (on_board yes) (dnp no) (fields_autoplaced)
+    (property "Reference" "#PWR023" (at 150.495 166.37 0)
+      (effects (font (size 1.27 1.27)) hide)
+    )
+    (property "Value" "GND" (at 150.495 164.4634 0)
+      (effects (font (size 1.27 1.27)))
+    )
+    (property "Footprint" "" (at 150.495 160.02 0)
+      (effects (font (size 1.27 1.27)) hide)
+    )
+    (property "Datasheet" "" (at 150.495 160.02 0)
+      (effects (font (size 1.27 1.27)) hide)
+    )
+    (pin "1")
+    (instances
+      (project "TVZ_KTM_ApplicationBoard"
+        (path "/e6e1ba2c-0a46-4bca-b3ad-33e778ea698b"
+          (reference "#PWR023") (unit 1)
+        )
+      )

Commit message: update
Connections:
- net I2C_SCL: now also TP5.1; no longer TP6.1
- net I2C_SDA: now also TP6.1; no longer TP5.1
Changed lines of the file:
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@@
     )
   )
-  (global_label "I2C_SCL" (shape input) (at 53.975 130.175 270) (fields_autoplaced)
+  (global_label "I2C_SCL" (shape input) (at 57.785 130.175 270) (fields_autoplaced)
     (effects (font (size 1.27 1.27)) (justify right))
-    (property "Intersheetrefs" "${INTERSHEET_REFS}" (at 53.975 140.7197 90)
+    (property "Intersheetrefs" "${INTERSHEET_REFS}" (at 57.785 140.7197 90)
       (effects (font (size 1.27 1.27)) (justify right) hide)
     )
@@
     )
   )
-  (global_label "I2C_SDA" (shape input) (at 57.785 130.175 270) (fields_autoplaced)
+  (global_label "I2C_SDA" (shape input) (at 53.975 130.175 270) (fields_autoplaced)
     (effects (font (size 1.27 1.27)) (justify right))
-    (property "Intersheetrefs" "${INTERSHEET_REFS}" (at 57.785 140.7802 90)
+    (property "Intersheetrefs" "${INTERSHEET_REFS}" (at 53.975 140.7802 90)
       (effects (font (size 1.27 1.27)) (justify right) hide)
     )

Commit message: update
Connections:
- net +5V: no longer C3.1, U3.3 (VDD)
- net GND: no longer TP14.1
- new net DAC(S): TP14.1
- new net VDD: C3.1, U3.3 (VDD)
Other:
- note added: "TODO: - provjeriti TP14 (jel treba DAC slave?) - LED13 nije spojena, čemu ono služi? (mislim da je za DAC slave?)"
- note removed: "TODO: - obratiti pozornost na MSB i LSB kod rasporeda sklopki, LEDica i ostalih elemenata - provjeriti TP14 (jel treba DAC slave?) - MCP2551 naponsko djelilo ( RX na 3.3V?) - LED13 nije spojena, čemu ono služi? (mislim da je za DAC slave?) - sitotisak pinovi"
Changed lines of the file:
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@@
     (effects (font (size 2.54 2.54) (thickness 0.508) bold) (justify left bottom))
   )
-  (text "TODO:\n- obratiti pozornost na MSB i LSB kod rasporeda sklopki, LEDica i ostalih elemenata\n- provjeriti TP14 (jel treba DAC slave?)\n- MCP2551 naponsko djelilo ( RX na 3.3V?)\n- LED13 nije spojena, čemu ono služi? (mislim da je za DAC slave?)\n- sitotisak pinovi"
+  (text "TODO:\n- provjeriti TP14 (jel treba DAC slave?)\n- LED13 nije spojena, čemu ono služi? (mislim da je za DAC slave?)"
     (at 15.875 191.77 0)
     (effects (font (size 1.27 1.27)) (justify left bottom))
@@
     )
   )
+  (global_label "DAC(S)" (shape input) (at 150.495 160.02 270) (fields_autoplaced)
+    (effects (font (size 1.27 1.27)) (justify right))
+    (property "Intersheetrefs" "${INTERSHEET_REFS}" (at 150.495 169.5367 90)
+      (effects (font (size 1.27 1.27)) (justify right) hide)
+    )
+  )
   (global_label "CAN_TD(M)" (shape input) (at 181.61 111.76 180) (fields_autoplaced)
     (effects (font (size 1.27 1.27)) (justify right))
@@
         (path "/e6e1ba2c-0a46-4bca-b3ad-33e778ea698b"
           (reference "C1") (unit 1)
-        )
-      )
-    )
-  )
-  (symbol (lib_name "GND_29") (lib_id "power:GND") (at 150.495 160.02 0) (unit 1)
-    (in_bom yes) (on_board yes) (dnp no) (fields_autoplaced)
-    (property "Reference" "#PWR023" (at 150.495 166.37 0)
-      (effects (font (size 1.27 1.27)) hide)
-    )
-    (property "Value" "GND" (at 150.495 164.4634 0)
-      (effects (font (size 1.27 1.27)))
-    )
-    (property "Footprint" "" (at 150.495 160.02 0)
-      (effects (font (size 1.27 1.27)) hide)
-    )
-    (property "Datasheet" "" (at 150.495 160.02 0)
-      (effects (font (size 1.27 1.27)) hide)
-    )
-    (pin "1")
-    (instances
-      (project "TVZ_KTM_ApplicationBoard"
-        (path "/e6e1ba2c-0a46-4bca-b3ad-33e778ea698b"
-          (reference "#PWR023") (unit 1)
         )
       )
@@
     )
   )
+  (symbol (lib_id "power:VDD") (at 241.935 104.14 0) (unit 1)
+    (in_bom yes) (on_board yes) (dnp no) (fields_autoplaced)
+    (property "Reference" "#PWR026" (at 241.935 107.95 0)
+      (effects (font (size 1.27 1.27)) hide)
+    )
+    (property "Value" "VDD" (at 241.935 100.0069 0)
+      (effects (font (size 1.27 1.27)))
+    )
+    (property "Footprint" "" (at 241.935 104.14 0)
+      (effects (font (size 1.27 1.27)) hide)
+    )
+    (property "Datasheet" "" (at 241.935 104.14 0)
+      (effects (font (size 1.27 1.27)) hide)
+    )
+    (pin "1")
+    (instances
+      (project "TVZ_KTM_ApplicationBoard"
+        (path "/e6e1ba2c-0a46-4bca-b3ad-33e778ea698b"
+          (reference "#PWR026") (unit 1)
+        )
+      )
+    )
+  )
   (symbol (lib_name "GND_9") (lib_id "power:GND") (at 239.395 23.495 0) (unit 1)
     (in_bom yes) (on_board yes) (dnp no) (fields_autoplaced)
@@
         )
       )
-    )
-  )
-  (symbol (lib_id "power:+5V") (at 241.935 104.14 0) (unit 1)
-    (in_bom yes) (on_board yes) (dnp no) (fields_autoplaced)
-    (property "Reference" "#PWR026" (at 241.935 107.95 0)
-      (effects (font (size 1.27 1.27)) hide)
-    )
-    (property "Value" "+5V" (at 241.935 100.5642 0)
-      (effects (font (size 1.27 1.27)))
-    )
-    (property "Footprint" "" (at 241.935 104.14 0)
-      (effects (font (size 1.27 1.27)) hide)
-    )
-    (property "Datasheet" "" (at 241.935 104.14 0)
-      (effects (font (size 1.27 1.27)) hide)
-    )
-    (pin "1")
-    (instances
-      (project "TVZ_KTM_ApplicationBoard"
-        (path "/e6e1ba2c-0a46-4bca-b3ad-33e778ea698b"
-          (reference "#PWR026") (unit 1)
-        )
-      )

Commit message: update
Changed lines of the file:
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@@
+    )
+  )
+  (symbol (lib_id "power:VDD") (at 200.66 26.035 0) (unit 1)
+    (in_bom yes) (on_board yes) (dnp no) (fields_autoplaced)
+    (property "Reference" "#PWR023" (at 200.66 29.845 0)
+      (effects (font (size 1.27 1.27)) hide)
+    )
+    (property "Value" "VDD" (at 200.66 21.9019 0)
+      (effects (font (size 1.27 1.27)))
+    )
+    (property "Footprint" "" (at 200.66 26.035 0)
+      (effects (font (size 1.27 1.27)) hide)
+    )
+    (property "Datasheet" "" (at 200.66 26.035 0)
+      (effects (font (size 1.27 1.27)) hide)
+    )
+    (pin "1")
+    (instances
+      (project "TVZ_KTM_ApplicationBoard"
+        (path "/e6e1ba2c-0a46-4bca-b3ad-33e778ea698b"
+          (reference "#PWR023") (unit 1)
+        )
+      )
     )
   )
@@
         )
       )
+    )
+  )
+  (symbol (lib_id "power:PWR_FLAG") (at 200.66 26.035 180) (unit 1)
+    (in_bom yes) (on_board yes) (dnp no) (fields_autoplaced)
+    (property "Reference" "#FLG04" (at 200.66 27.94 0)
+      (effects (font (size 1.27 1.27)) hide)
+    )
+    (property "Value" "PWR_FLAG" (at 202.311 27.7388 0)
+      (effects (font (size 1.27 1.27)) (justify right))
+    )
+    (property "Footprint" "" (at 200.66 26.035 0)
+      (effects (font (size 1.27 1.27)) hide)
+    )
+    (property "Datasheet" "~" (at 200.66 26.035 0)
+      (effects (font (size 1.27 1.27)) hide)
+    )
+    (pin "1")
+    (instances
+      (project "TVZ_KTM_ApplicationBoard"
+        (path "/e6e1ba2c-0a46-4bca-b3ad-33e778ea698b"
+          (reference "#FLG04") (unit 1)
+        )
+      )

Commit message: update
Other:
- moved on the sheet: C1, JP1, JP2, JP3, R1, R2, R3, R4, R5, TP5, TP6, U1

Commit message: v1rev1
Other:
- note removed: "TODO: - provjeriti TP14 (jel treba DAC slave?) - LED13 nije spojena, čemu ono služi? (mislim da je za DAC slave?)"
Changed lines of the file:
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@@
     (effects (font (size 2.54 2.54) (thickness 0.508) bold) (justify left bottom))
-  )
-  (text "TODO:\n- provjeriti TP14 (jel treba DAC slave?)\n- LED13 nije spojena, čemu ono služi? (mislim da je za DAC slave?)"
-    (at 15.875 191.77 0)
-    (effects (font (size 1.27 1.27)) (justify left bottom))
   )
   (text "BUSY" (at 107.95 175.26 0)

Commit message: update
Other:
- note added: "TODO: - LED PA15 premjestiti na PA9 u kicadu i brikati na testnoj pločici"
Changed lines of the file:
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@@
     (stroke (width 0) (type default))
+  )
+  (text "TODO:\n- LED PA15 premjestiti na PA9 u kicadu i brikati na testnoj pločici"
+    (at 25.4 177.165 0)
+    (effects (font (size 1.27 1.27)) (justify left bottom))
   )
   (text "CAN" (at 213.36 97.155 0)
