File: KiCAD files/TVZ_KTM_ApplicationBoard.kicad_pcb (KiCad board)
At the start: 2 copper layers, 146 x 55 mm, 114 parts, among them J1 Conn_02x19_Odd_Even, J2 Conn_02x19_Odd_Even, J3 Conn_02x19_Odd_Even, J4 Conn_02x19_Odd_Even, SW1 EG1271A, SW2 EG1271A, SW3 EG1271A, SW4 EG1271A, U1 LM75B, U2 MCP2551-I-P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

Commit message: update
Parts:
- removed G***: LOGO, Footprint:tvz3
- removed kibuzzard-63D0F0B6 (x2): G***, kibuzzard-63D0F0B6
- added TP15: TestPoint, Footprint:KEYS4952, F.Cu at (143.6, 106.6)
- J1, J2, J3, J4: footprint Connector_PinSocket_2.54mm:PinSocket_2x19_P2.54mm_Vertical_SMD -> Connector_PinSocket_2.54mm:PinSocket_2x19_P2.54mm_Vertical
- JP1, JP4, JP5: footprint Connector_PinHeader_2.54mm:PinHeader_1x03_P2.54mm_Vertical_SMD_Pin1Right -> Connector_PinHeader_2.54mm:PinHeader_1x03_P2.54mm_Vertical
- moved kibuzzard-64A69B51 69.3 mm to (69.9, 98.6)
- moved kibuzzard-64A69B71 69.3 mm to (75.9, 98.6)
- moved kibuzzard-64A69B81 69.3 mm to (81.9, 98.6)
- moved kibuzzard-64A69B8B 69.3 mm to (87.9, 98.6)
- moved TP6 54.2 mm to (70.0, 106.6)
- moved kibuzzard-63D0FB98 54.2 mm to (70.0, 103.1)
- moved J2 48.7 mm to (120.2, 61.2)
- moved J1 48.6 mm to (59.3, 61.2)
- moved U2 45.2 mm to (87.7, 74.1), turned to 90 degrees
- moved TP9 43.4 mm to (129.6, 106.6)
- moved C2 43.3 mm to (84.5, 69.2)
- moved D10 43.3 mm to (76.0, 95.2)
- moved D11 43.3 mm to (82.0, 95.2)
- moved D12 43.3 mm to (88.0, 95.2)
- moved D5 43.3 mm to (96.0, 95.2)
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Connections:
- R10 pad 1: PC0_1 -> PC6_1
- R11 pad 1: PC1_1 -> PC7_1
- R12 pad 1: PC2_1 -> PC8_1
- R13 pad 1: PC3_1 -> PC9_1
- R14 pad 1: PC6_1 -> PC0_1
- R15 pad 1: PC7_1 -> PC1_1
- R16 pad 1: PC8_1 -> PC2_1
- R17 pad 1: PC9_1 -> PC3_1
Routing:
- net PB7_1: track 0.00 -> 127.9 mm
- net PB9_1: track 4.14 -> 125.4 mm
- net PB8_1: track 4.53 -> 125.1 mm
- net PB3_SCK: track 0.00 -> 113.9 mm
- net PA10_1: track 132.0 -> 19.2 mm, vias 2 -> 0
- net PB14_1: track 0.00 -> 109.3 mm
- net PB13_1: track 0.00 -> 105.9 mm
- net PB15_1: track 0.00 -> 100.6 mm
- net /CANL: track 39.7 -> 109.2 mm
- net PB2_1: track 50.5 -> 0.00 mm, vias 1 -> 0
- net PB1_1: track 47.1 -> 0.00 mm, vias 1 -> 0
- net PA11_1: track 40.1 -> 0.00 mm, vias 1 -> 0
- net PA4_1: track 172.8 -> 211.5 mm, vias 2 -> 0
- net GND: track 37.9 -> 0.00 mm, vias 20 -> 0
- net +5V: track 34.8 -> 0.00 mm, vias 1 -> 0
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- removed copper zone on F.Cu, net GND
Other:
- board size 146 x 55 mm -> 161.7 x 59.5 mm
- board text removed: "TVZ.KTM.ApplicationBoard.v1rev1"

Commit message: update
Parts:
- moved U3 10.7 mm to (187.9, 65.2), turned to -90 degrees
- moved C2 1.32 mm to (84.2, 70.5)
Connections:
- J2 pad 32: unconnected-(J2-Pin_32-Pad32) -> GND
- J3 pad 16: +3V3 -> unconnected-(J3-Pin_16-Pad16)
- J4 pad 32: unconnected-(J4-Pin_32-Pad32) -> GND
Routing:
- net PA7_BUSY: track 0.00 -> 201.3 mm, vias 0 -> 2
- net +5V: track 0.00 -> 180.6 mm, vias 0 -> 3
- net PA8_STROBE: track 0.00 -> 168.3 mm
- net PA10_1: track 19.2 -> 175.6 mm
- net +3V3: track 4.39 -> 139.7 mm, vias 0 -> 7
- net PB8_1: track 125.1 -> 229.0 mm
- net PC6_2: track 0.00 -> 97.0 mm, vias 0 -> 2
- net PC8_2: track 0.00 -> 93.5 mm
- net PC3_1: track 0.00 -> 93.4 mm
- net PB9_1: track 125.4 -> 217.7 mm
- net PC2_1: track 0.00 -> 77.0 mm
- net PA11_2: track 0.00 -> 64.1 mm
- net PC7_2: track 0.00 -> 55.6 mm, vias 0 -> 6
- net PC1_1: track 0.00 -> 54.5 mm
- net PB2_1: track 0.00 -> 53.3 mm, vias 0 -> 3
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Other:
- board outline removed

Commit message: update
Parts:
- removed J1, J2, J3, J4: Conn_02x19_Odd_Even, Connector_PinSocket_2.54mm:PinSocket_2x19_P2.54mm_Vertical
- removed JP4, JP5: Jumper_3_Open, Connector_PinHeader_2.54mm:PinHeader_1x03_P2.54mm_Vertical
- removed kibuzzard-63D0FC24: G***, kibuzzard-63D0FC24
- removed kibuzzard-63D0FC34: G***, kibuzzard-63D0FC34
- removed kibuzzard-63D0FC3F: G***, kibuzzard-63D0FC3F
- removed kibuzzard-63D0FC48: G***, kibuzzard-63D0FC48
- removed kibuzzard-63D12AAF (x2): G***, kibuzzard-63D12AAF
- removed kibuzzard-63D12AD6 (x2): G***, kibuzzard-63D12AD6
- removed kibuzzard-63D12AE3 (x2): G***, kibuzzard-63D12AE3
- removed kibuzzard-63D12AEC (x2): G***, kibuzzard-63D12AEC
- removed kibuzzard-63E0EDBE: G***, kibuzzard-63E0EDBE
- removed kibuzzard-64A69B51: G***, kibuzzard-64A69B51
- removed kibuzzard-64A69B71: G***, kibuzzard-64A69B71
- removed kibuzzard-64A69B81: G***, kibuzzard-64A69B81
- removed kibuzzard-64A69B8B: G***, kibuzzard-64A69B8B
- added JP2: Jumper_3_Open, Connector_PinHeader_2.54mm:PinHeader_1x03_P2.54mm_Vertical, F.Cu at (120.0, 47.4)
- added JP3: Jumper_3_Open, Connector_PinHeader_2.54mm:PinHeader_1x03_P2.54mm_Vertical, F.Cu at (115.3, 47.4)
- added U4: NUCLEO64-F446RE, Footprint:NUCLEO64, F.Cu at (43.6, 37.1)
- added U5: NUCLEO64-F446RE, Footprint:NUCLEO64, F.Cu at (140.3, 37.8)
- moved kibuzzard-63D0FBC8 68.0 mm to (70.0, 79.7), turned to 90 degrees
- moved TP15 64.9 mm to (84.3, 80.4)
- moved TP9 59.7 mm to (76.1, 80.2)
- moved TP5 58.2 mm to (127.1, 71.2)
- moved TP6 58.2 mm to (116.1, 71.2)
- moved kibuzzard-63D0FB98 58.2 mm to (116.1, 67.7)
- moved kibuzzard-63D0FBA8 58.2 mm to (127.1, 67.7)
- moved kibuzzard-63D26251 58.2 mm to (111.6, 69.6)
- moved kibuzzard-63D262D2 46.2 mm to (49.5, 79.6)
- moved TP7 46.2 mm to (64.5, 81.2)
- moved TP8 46.2 mm to (53.5, 81.2)
- moved kibuzzard-63D0FBB4 46.2 mm to (64.5, 77.7)
- moved kibuzzard-63D0FBBC 46.2 mm to (53.5, 77.7)
- moved R1 30.2 mm to (113.5, 53.2)
- moved R2 30.2 mm to (113.5, 57.0)
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Connections:
- R1 pad 1: PB8_1 -> I2C_SCL
- R10 pad 1: PC6_1 -> LED5(M)
- R11 pad 1: PC7_1 -> LED6(M)
- R12 pad 1: PC8_1 -> LED7(M)
- R13 pad 1: PC9_1 -> LED8(M)
- R14 pad 1: PC0_1 -> LED1(M)
- R15 pad 1: PC1_1 -> LED2(M)
- R16 pad 1: PC2_1 -> LED3(M)
- R17 pad 1: PC3_1 -> LED4(M)
- R2 pad 1: PB9_1 -> I2C_SDA
- R20 pad 1: PA4_2 -> unconnected-(R20-Pad1)
- R6 pad 1: PC6_2 -> LED1(S)
- R7 pad 1: PC7_2 -> LED2(S)
- R8 pad 1: PC8_2 -> LED3(S)
- R9 pad 1: PC9_2 -> LED4(S)
- SW1 pad 2: PB0_1 -> S1
- SW2 pad 2: PB1_1 -> S2
- SW3 pad 2: PB2_1 -> S3
- SW4 pad 2: PB10_1 -> S4
- TP12 pad 1: PB4_MISO -> SPI_MISO
- TP13 pad 1: PB5_MOSI -> SPI_MOSI
- TP2 pad 1: PA4_1 -> DAC(M)>>ADC(S)
- TP5 pad 1: PB9_1 -> I2C_SCL
- TP6 pad 1: PB8_1 -> I2C_SDA
- TP7 pad 1: PA10_1 -> USART_TX(M) >> USART_RX(S)
- TP8 pad 1: PA9_1 -> USART_RX(M) >> USART_TX(S)
- U1 pad 1: PB9_1 -> I2C_SDA
- U1 pad 2: PB8_1 -> I2C_SCL
- U2 pad 1: PA12_1 -> CAN_TD(M)
- U2 pad 4: PA11_1 -> CAN_RD(M)
- U3 pad 1: PA12_2 -> CAN_TD(S)
- U3 pad 4: PA11_2 -> CAN_RD(S)
Routing:
- net PA4_1: track 236.7 -> 0.00 mm
- net PB8_1: track 229.0 -> 0.00 mm
- net USART_TX(M) >> USART_RX(S): track 0.00 -> 221.1 mm
- net PB9_1: track 217.7 -> 0.00 mm
- net PA7_BUSY: track 201.3 -> 0.00 mm, vias 2 -> 0
- net USART_RX(M) >> USART_TX(S): track 0.00 -> 195.1 mm
- net PA10_1: track 175.6 -> 0.00 mm
- net PA8_STROBE: track 168.3 -> 0.00 mm
- net I2C_SDA: track 0.00 -> 166.6 mm
- net I2C_SCL: track 0.00 -> 153.8 mm
- net +5V: track 180.6 -> 38.3 mm, vias 3 -> 0
- net PB7_1: track 136.6 -> 0.00 mm
- net +3V3: track 139.7 -> 4.65 mm, vias 7 -> 0
- net SPI_MOSI: track 0.00 -> 132.8 mm
- net SPI_MISO: track 0.00 -> 117.6 mm
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- removed copper zone on B.Cu, net GND

Commit message: update
Parts:
- removed kibuzzard-63D0FBB4: G***, kibuzzard-63D0FBB4
- removed kibuzzard-63D0FBBC: G***, kibuzzard-63D0FBBC
- removed kibuzzard-63D0FBC8: G***, kibuzzard-63D0FBC8
- removed kibuzzard-63D12B8B (x2): G***, kibuzzard-63D12B8B
- removed kibuzzard-63D13186: G***, kibuzzard-63D13186
- removed the kibuzzard-63D255AB at (49.5, 44.0)
- removed kibuzzard-63D262D2: G***, kibuzzard-63D262D2
- removed the kibuzzard-63D26411 at (89.9, 43.6)
- moved C2 3.35 mm to (67.6, 41.7)
- moved TP2 3.11 mm to (97.1, 78.3)
- moved U2 3.11 mm to (71.6, 45.5)
- moved TP8 2.90 mm to (53.6, 78.3)
- moved TP7 2.90 mm to (64.5, 78.3)
- moved TP15 2.84 mm to (86.2, 78.3)
- moved D5 2.64 mm to (79.1, 67.2)
- moved D6 2.64 mm to (85.1, 67.2)
- moved D7 2.64 mm to (91.1, 67.2)
- moved D8 2.64 mm to (97.1, 67.2)
- moved R10 2.64 mm to (79.1, 64.2)
- moved R11 2.64 mm to (85.1, 64.2)
- moved R12 2.64 mm to (91.1, 64.2)
- moved R13 2.64 mm to (97.1, 64.2)
- moved D11 2.53 mm to (65.6, 67.2)
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Connections:
- TP10 pad 1: PA7_BUSY -> BUSY
- TP11 pad 1: PA8_STROBE -> STROBE
- TP14 pad 1: PA4_2 -> unconnected-(TP14-Pad1)
- TP7 pad 1: USART_TX(M) >> USART_RX(S) -> USART_RX(M) >> USART_TX(S)
- TP8 pad 1: USART_RX(M) >> USART_TX(S) -> USART_TX(M) >> USART_RX(S)
- U4 pad 35: unconnected-(U4-PC2-Pad35) -> BUSY
- U4 pad 37: unconnected-(U4-PC3-Pad37) -> STROBE
- U4 pad 67: unconnected-(U4-PB5-Pad67) -> D1
- U4 pad 68: unconnected-(U4-PB13-Pad68) -> D4
- U4 pad 71: unconnected-(U4-PA10-Pad71) -> D2
- U4 pad 72: unconnected-(U4-PC4-Pad72) -> D3
- U5 pad 30: unconnected-(U5-PA1-Pad30) -> STROBE
- U5 pad 32: unconnected-(U5-PA4-Pad32) -> BUSY
- U5 pad 34: unconnected-(U5-PB0-Pad34) -> D4
- U5 pad 35: unconnected-(U5-PC2-Pad35) -> D3
- U5 pad 36: unconnected-(U5-PC1-Pad36) -> D2
- U5 pad 37: unconnected-(U5-PC3-Pad37) -> D1
Routing:
- net USART_TX(M) >> USART_RX(S): track 221.1 -> 0.00 mm
- net USART_RX(M) >> USART_TX(S): track 195.1 -> 0.00 mm
- net I2C_SDA: track 166.6 -> 0.00 mm
- net I2C_SCL: track 153.8 -> 0.00 mm
- net SPI_MOSI: track 132.8 -> 0.00 mm
- net /CANH: track 131.2 -> 0.00 mm
- net SPI_MISO: track 117.6 -> 0.00 mm
- net /CANL: track 110.5 -> 0.00 mm
- net CAN_RD(S): track 92.5 -> 0.00 mm
- net SPI_~{CS}: track 86.4 -> 0.00 mm
- net DAC(M)>>ADC(S): track 86.2 -> 0.00 mm
- net SPI_SCK: track 74.7 -> 0.00 mm
- net CAN_TD(S): track 70.3 -> 0.00 mm
- net LED1(S): track 62.1 -> 0.00 mm
- net LED8(M): track 61.0 -> 0.00 mm
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Other:
- board outline added: 186 x 63.6 mm
- board text added: "DAC"
- board text added: "GND"
- board text added: "LED"
- board text added: "LED1"
- board text added: "LED2"
- board text added: "LED3"
- board text added: "LED4"
- board text added: "LED5"
- board text added: "LED6"
- board text added: "LED7"
- board text added: "LED8"
- board text added: "MASTER"
- board text added: "MCP2551"
- board text added: "PA0"
- board text added: "PA1"
- board text added: "PA15"
- board text added: "PA4"
- board text added: "PA5"
- board text added: "PA6"
- board text added: "PA7"
- board text added: "PB0"
- board text added: "PB6"
- board text added: "PB7"
- board text added: "PC0"
- board text added: "PC1"
- board text added: "PC13"
- board text added: "PC14"
- board text added: "PC7"
- board text added: "RESET"
- board text added: "RX"
- board text added: "S1"
- board text added: "S2"
- board text added: "S3"
- board text added: "S4"
- board text added: "SKLOPKE"
- board text added: "TX"
- board text added: "USER"

Commit message: update
Parts:
- removed kibuzzard-63D0FB98: G***, kibuzzard-63D0FB98
- removed kibuzzard-63D0FBA8: G***, kibuzzard-63D0FBA8
- removed kibuzzard-63D0FCA0: G***, kibuzzard-63D0FCA0
- removed kibuzzard-63D0FCA9: G***, kibuzzard-63D0FCA9
- removed kibuzzard-63D121CA: G***, kibuzzard-63D121CA
- removed kibuzzard-63D12226: G***, kibuzzard-63D12226
- removed kibuzzard-63D12234: G***, kibuzzard-63D12234
- removed kibuzzard-63D1223E: G***, kibuzzard-63D1223E
- removed kibuzzard-63D123B4: G***, kibuzzard-63D123B4
- removed kibuzzard-63D255AB: G***, kibuzzard-63D255AB
- removed kibuzzard-63D25AA1: G***, kibuzzard-63D25AA1
- removed kibuzzard-63D26251: G***, kibuzzard-63D26251
- removed kibuzzard-63D26411: G***, kibuzzard-63D26411
- removed kibuzzard-63D26434: G***, kibuzzard-63D26434
- removed kibuzzard-63D2644E: G***, kibuzzard-63D2644E
- removed kibuzzard-63D26457: G***, kibuzzard-63D26457
- removed kibuzzard-63E0EC18: G***, kibuzzard-63E0EC18
- removed kibuzzard-63E0EE4D: G***, kibuzzard-63E0EE4D
- removed kibuzzard-63E123CE: G***, kibuzzard-63E123CE
- removed kibuzzard-63E123D9: G***, kibuzzard-63E123D9
- removed kibuzzard-648ABAA6: G***, kibuzzard-648ABAA6
- moved TP13 11.6 mm to (155.0, 77.6)
- moved TP4 11.1 mm to (162.6, 65.4)
- moved TP10 11.0 mm to (183.5, 77.9)
- moved C1 10.8 mm to (118.5, 49.5), turned to 180 degrees
- moved TP12 10.7 mm to (142.0, 77.3)
- moved TP14 10.7 mm to (177.0, 65.5)
- moved U3 10.2 mm to (166.9, 37.9)
- moved D1 10.0 mm to (141.7, 56.6)
- moved D13 10.0 mm to (183.6, 56.6)
- moved D3 10.0 mm to (159.8, 56.6)
- moved D4 10.0 mm to (168.9, 56.6)
- moved R20 10.0 mm to (183.6, 53.5)
- moved R7 10.0 mm to (150.7, 53.5)
- moved R8 10.0 mm to (159.8, 53.5)
- moved D2 10.0 mm to (150.8, 56.6)
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Connections:
- TP5 pad 1: I2C_SCL -> I2C_SDA
- TP6 pad 1: I2C_SDA -> I2C_SCL
Routing:
- net I2C_SDA: track 0.00 -> 111.8 mm
- net /CANH: track 0.00 -> 111.1 mm
- net /CANL: track 0.00 -> 99.5 mm
- net I2C_SCL: track 0.00 -> 96.9 mm
- net SPI_~{CS}: track 0.00 -> 78.0 mm
- net DAC(M)>>ADC(S): track 0.00 -> 77.9 mm
- net SPI_MISO: track 0.00 -> 65.1 mm
- net SPI_SCK: track 0.00 -> 58.0 mm
- net SPI_MOSI: track 0.00 -> 56.9 mm
- net S1: track 0.00 -> 53.3 mm
- net D1: track 0.00 -> 41.7 mm
- net S3: track 0.00 -> 40.6 mm
- net Net-(JP3-C): track 0.00 -> 38.8 mm
- net CAN_TD(M): track 0.00 -> 37.3 mm
- net CAN_RD(M): track 0.00 -> 36.5 mm
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Other:
- board size 186 x 63.6 mm -> 160 x 58.3 mm
- board text added: "A0"
- board text added: "A1"
- board text added: "A2"
- board text added: "BUSY"
- board text added: "CAN"
- board text added: "CANH"
- board text added: "CANL"
- board text added: "I2C"
- board text added: "LM75B"
- board text added: "MISO"
- board text added: "MOSI"
- board text added: "PAR.KOM."
- board text added: "PB9"
- board text added: "PC6"
- board text added: "SCL"
- board text added: "SDA"
- board text added: "SLAVE"
- board text added: "SPI"
- board text added: "STROBE"
- board text added: "UART"

Commit message: update
Parts:
- moved TP3 2.13 mm to (148.3, 65.9)
- moved D13 1.80 mm to (184.2, 54.9)
- moved D1 1.72 mm to (142.0, 54.9)
- moved D2 1.72 mm to (151.0, 54.9)
- moved D3 1.71 mm to (160.0, 54.9)
- moved D4 1.71 mm to (169.1, 54.9)
- moved R20 1.65 mm to (184.2, 51.9)
- moved R6 1.58 mm to (142.0, 51.9)
- moved R7 1.58 mm to (151.0, 51.9)
- moved R8 1.57 mm to (160.1, 51.9)
- moved R9 1.57 mm to (169.1, 51.9)
- moved TP10 1.45 mm to (184.9, 78.3)
- moved TP11 1.28 mm to (170.4, 78.3)
- moved TP12 1.16 mm to (141.3, 78.3)
- moved TP13 1.08 mm to (155.8, 78.3)
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Connections:
- R20 pad 1: unconnected-(R20-Pad1) -> DAC(M)>>ADC(S)
- TP14 pad 1: unconnected-(TP14-Pad1) -> GND
Routing:
- net USART_TX(M) >> USART_RX(S): track 0.00 -> 224.0 mm
- net USART_RX(M) >> USART_TX(S): track 0.00 -> 202.8 mm
- net BUSY: track 0.00 -> 174.6 mm
- net STROBE: track 0.00 -> 147.2 mm
- net CAN_RD(S): track 0.00 -> 87.3 mm
- net CAN_TD(S): track 0.00 -> 69.6 mm
- net LED8(M): track 0.00 -> 68.6 mm
- net LED7(M): track 0.00 -> 65.5 mm
- net LED1(S): track 0.00 -> 63.2 mm
- net SPI_MOSI: track 56.9 -> 117.9 mm
- net LED6(M): track 0.00 -> 55.4 mm
- net LED2(S): track 0.00 -> 50.0 mm
- net LED5(M): track 0.00 -> 48.1 mm
- net LED3(S): track 0.00 -> 43.6 mm
- net +5V: track 10.3 -> 52.7 mm
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- added copper zone on B.Cu, net GND
Other:
- board size 160 x 58.3 mm -> 160 x 59.6 mm
- board text added: "PA11"
- board text added: "PA12"
- board text added: "PB14/PC11"
- board text added: "PB15/PC12"
- board text added: "PC2/PA4"
- board text added: "PC3/PA1"
- board text removed: "USER"

Commit message: update
Parts:
- moved C1 0.20 mm to (118.5, 49.3)
Connections:
- TP5 pad 1: I2C_SDA -> I2C_SCL
- TP6 pad 1: I2C_SCL -> I2C_SDA
Routing:
- net I2C_SCL: track 128.5 -> 145.8 mm
- net GND: track 13.2 -> 23.9 mm, vias 9 -> 17
- net +3V3: track 10.9 -> 19.9 mm
- net I2C_SDA: track 149.6 -> 157.1 mm
- net Net-(JP3-C): track 38.8 -> 44.4 mm
- net D4: track 33.6 -> 30.0 mm
- net unconnected-(SW1-A-Pad1): track 0.00 -> 3.20 mm
- net unconnected-(SW4-A-Pad1): track 0.00 -> 3.20 mm
- net unconnected-(SW3-A-Pad1): track 0.00 -> 3.20 mm
- net unconnected-(SW2-A-Pad1): track 0.00 -> 3.20 mm
- net USART_TX(M) >> USART_RX(S): track 224.0 -> 226.3 mm
- net LED3(S): track 43.6 -> 42.0 mm
- net CAN_RD(S): track 87.3 -> 88.9 mm
- net +5V: track 52.7 -> 53.9 mm, vias 0 -> 1
- net CAN_TD(S): track 69.6 -> 70.8 mm
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Other:
- board size 160 x 59.6 mm -> 160 x 60 mm
