File: KiCAD files/TVZ_KTM_ApplicationBoard.kicad_pcb (KiCad board)
At the start: 2 copper layers, 160 x 60 mm, 63 parts, among them SW1 EG1271A, SW2 EG1271A, SW3 EG1271A, SW4 EG1271A, U1 LM75B, U2 MCP2551-I-P, U3 MCP2551-I-P, U4 NUCLEO64-F446RE, U5 NUCLEO64-F446RE

Commit message: update
Connections:
- U4 pad 25: LED1(M) -> unconnected-(U4-PC14-Pad25)
- U4 pad 39: unconnected-(U4-PC9-Pad39) -> LED1(M)
Routing:
- net LED1(M): track 10.5 -> 112.7 mm
- net I2C_SDA: track 157.1 -> 150.7 mm
Other:
- board text added: "PC9"
- board text removed: "PC14"

Commit message: update
Connections:
- U4 pad 17: LED5(M) -> unconnected-(U4-PA15-Pad17)
- U4 pad 51: LED6(M) -> LED5(M)
- U4 pad 53: LED7(M) -> LED6(M)
- U4 pad 59: unconnected-(U4-PA9-Pad59) -> LED8(M)
- U4 pad 61: LED8(M) -> LED7(M)
Routing:
- net DAC(M)>>ADC(S): track 84.3 -> 77.0 mm
- net LED8(M): track 10.9 -> 15.7 mm
- net LED7(M): track 20.5 -> 17.3 mm, vias 0 -> 1
- net LED5(M): track 37.4 -> 34.4 mm
- net S4: track 17.6 -> 15.5 mm
- net LED6(M): track 28.1 -> 26.5 mm
Other:
- board text added: "PA9"
- board text added: "TVZ KTM Application board v1rev2"
- board text removed: "PA15"
- board text removed: "TVZ KTM Application board v1rev1"

Commit message: update
Connections:
- U4 pad 23: LED2(M) -> LED4(M)
- U4 pad 36: LED3(M) -> LED2(M)
- U4 pad 38: LED4(M) -> LED1(M)
- U4 pad 39: LED1(M) -> LED3(M)
Routing:
- net LED3(M): track 45.9 -> 131.2 mm
- net LED2(M): track 17.4 -> 62.7 mm
- net LED1(M): track 112.7 -> 75.8 mm
- net LED4(M): track 46.2 -> 37.6 mm
- net USART_TX(M) >> USART_RX(S): track 226.3 -> 225.7 mm

Commit message: update
Connections:
- U4 pad 23: LED4(M) -> unconnected-(U4-PC13-Pad23)
- U4 pad 39: LED3(M) -> LED4(M)
- U4 pad 40: unconnected-(U4-PC8-Pad40) -> LED3(M)
- U5 pad 51: LED3(S) -> LED1(S)
- U5 pad 52: LED2(S) -> LED3(S)
- U5 pad 53: LED1(S) -> LED2(S)
Routing:
- net LED4(M): track 37.6 -> 139.6 mm
- net LED2(S): track 52.2 -> 46.8 mm
- net LED1(S): track 58.7 -> 62.7 mm
- net LED3(S): track 39.4 -> 43.2 mm
- net LED3(M): track 131.2 -> 134.2 mm, vias 0 -> 4
- net I2C_SCL: track 145.8 -> 147.2 mm
Other:
- outline, holes or cut-outs redrawn
- board text added: "PC8"

Commit message: update
Connections:
- U4 pad 3: S1 -> S4
- U4 pad 57: S4 -> S1
Routing:
- net S4: track 15.5 -> 68.7 mm
- net S1: track 24.8 -> 62.4 mm, vias 0 -> 1
- net LED1(M): track 75.8 -> 73.1 mm
- net LED2(M): track 62.7 -> 61.5 mm

Commit message: update
Connections:
- U4 pad 60: unconnected-(U4-PB2-Pad60) -> D2
- U4 pad 62: unconnected-(U4-PB1-Pad62) -> D1
- U4 pad 65: unconnected-(U4-PB4-Pad65) -> D3
- U4 pad 67: D1 -> D4
- U4 pad 68: D4 -> unconnected-(U4-PB13-Pad68)
- U4 pad 71: D2 -> unconnected-(U4-PA10-Pad71)
- U4 pad 72: D3 -> unconnected-(U4-PC4-Pad72)
- U5 pad 34: D4 -> DAC(M)>>ADC(S)
- U5 pad 37: D1 -> D4
- U5 pad 38: DAC(M)>>ADC(S) -> D1
Routing:
- net D1: track 42.0 -> 0.00 mm
- net D2: track 33.3 -> 0.00 mm
- net D4: track 30.0 -> 0.00 mm
- net D3: track 26.9 -> 0.00 mm
- net DAC(M)>>ADC(S): track 77.0 -> 85.2 mm
- net BUSY: track 175.7 -> 177.1 mm
- net STROBE: track 146.8 -> 147.7 mm

Commit message: update
Connections:
- U4 pad 1: S2 -> S3
- U4 pad 2: S3 -> S2
- U4 pad 3: S4 -> S1
- U4 pad 36: LED2(M) -> LED3(M)
- U4 pad 38: LED1(M) -> LED4(M)
- U4 pad 39: LED4(M) -> LED1(M)
- U4 pad 40: LED3(M) -> LED2(M)
- U4 pad 51: LED5(M) -> LED8(M)
- U4 pad 53: LED6(M) -> LED7(M)
- U4 pad 57: S1 -> S4
- U4 pad 59: LED8(M) -> LED5(M)
- U4 pad 60: D2 -> D1
- U4 pad 61: LED7(M) -> LED6(M)
- U4 pad 62: D1 -> D2
- U4 pad 65: D3 -> D0
- U4 pad 67: D4 -> D3
- U5 pad 35: D3 -> D2
- U5 pad 36: D2 -> D0
- U5 pad 37: D4 -> D3
- U5 pad 50: LED4(S) -> LED1(S)
- U5 pad 51: LED1(S) -> LED4(S)
- U5 pad 52: LED3(S) -> LED2(S)
- U5 pad 53: LED2(S) -> LED3(S)
Routing:
- net LED3(M): track 134.2 -> 48.0 mm, vias 4 -> 0
- net LED4(M): track 139.6 -> 53.6 mm
- net D1: track 0.00 -> 59.4 mm
- net LED2(M): track 61.5 -> 118.3 mm, vias 0 -> 4
- net S4: track 68.7 -> 15.5 mm
- net LED1(M): track 73.1 -> 110.5 mm
- net D3: track 0.00 -> 37.2 mm
- net D0: track 0.00 -> 36.9 mm
- net S1: track 62.4 -> 25.7 mm, vias 1 -> 0
- net D2: track 0.00 -> 36.6 mm, vias 0 -> 2
- net LED8(M): track 15.7 -> 44.3 mm, vias 1 -> 0
- net S3: track 46.8 -> 58.6 mm
- net LED6(M): track 26.7 -> 34.3 mm, vias 0 -> 1
- net LED5(M): track 33.6 -> 28.8 mm, vias 0 -> 3
- net LED2(S): track 46.8 -> 51.4 mm
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Other:
- board text added: "LSB"
- board text added: "MSB"
- board text removed: "LED1"
- board text removed: "LED2"
- board text removed: "LED3"
- board text removed: "LED4"
- board text removed: "LED5"
- board text removed: "LED6"
- board text removed: "LED7"
- board text removed: "LED8"
- board text removed: "S1"
- board text removed: "S2"
- board text removed: "S3"
- board text removed: "S4"

Commit message: update
Connections:
- U4 pad 41: unconnected-(U4-PB8-Pad41) -> I2C_SCL
- U4 pad 42: I2C_SCL -> unconnected-(U4-PC6-Pad42)
Routing:
- net I2C_SDA: track 150.3 -> 155.2 mm
- net I2C_SCL: track 147.2 -> 149.6 mm
