File: KiCAD files/Master.kicad_sch (KiCad schematic)
At the start: 24 parts, among them SW1 EG1271A, SW2 EG1271A, SW3 EG1271A, SW4 EG1271A, U4 NUCLEO64-F446RE

Commit message: update
Connections:
- net BUSY: now reaches U4.35 (PC2)
- net STROBE: now reaches U4.37 (PC3)
- net D1: now reaches U4.67 (PB5)
- net D4: now reaches U4.68 (PB13)
- net D2: now reaches U4.71 (PA10)
- net D3: now reaches U4.72 (PC4)
- no-connect marks 40 -> 34
Changed lines of the file:
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@@
   )
   (no_connect (at 169.545 73.66))
-  (no_connect (at 113.665 101.6))
+  (no_connect (at 169.545 106.68))
   (no_connect (at 57.785 136.525))
   (no_connect (at 113.665 53.34))
-  (no_connect (at 169.545 76.2))
   (no_connect (at 113.665 116.84))
   (no_connect (at 113.665 106.68))
@@
   (no_connect (at 169.545 116.84))
   (no_connect (at 113.665 83.82))
-  (no_connect (at 113.665 99.06))
-  (no_connect (at 113.665 104.14))
   (no_connect (at 169.545 88.9))
   (no_connect (at 57.785 147.32))
@@
   (no_connect (at 169.545 104.14))
   (no_connect (at 139.065 40.64))
-  (no_connect (at 169.545 106.68))
   (no_connect (at 58.42 125.73))
   (no_connect (at 169.545 60.96))
@@
   (no_connect (at 144.145 40.64))
   (no_connect (at 131.445 40.64))
-  (no_connect (at 169.545 78.74))
   (no_connect (at 169.545 101.6))
   (no_connect (at 169.545 58.42))
@@
   (no_connect (at 128.905 40.64))
   (no_connect (at 113.665 88.9))
-  (no_connect (at 169.545 127))
+  (no_connect (at 169.545 99.06))
   (no_connect (at 113.665 132.08))
-  (no_connect (at 169.545 99.06))
+  (no_connect (at 169.545 76.2))
   (no_connect (at 126.365 40.64))
   (no_connect (at 169.545 86.36))
   (no_connect (at 113.665 114.3))
-  (no_connect (at 169.545 109.22))
   (no_connect (at 141.605 40.64))
   (wire (pts (xy 39.37 43.18) (xy 39.37 43.815))
@@
     )
   )
+  (global_label "D4" (shape input) (at 169.545 127 0) (fields_autoplaced)
+    (effects (font (size 1.27 1.27)) (justify left))
+    (property "Intersheetrefs" "${INTERSHEET_REFS}" (at 175.0097 127 0)
+      (effects (font (size 1.27 1.27)) (justify left) hide)
+    )
+  )
   (global_label "SPI_MISO" (shape input) (at 140.97 168.91 270) (fields_autoplaced)
     (effects (font (size 1.27 1.27)) (justify right))
@@
     )
   )
+  (global_label "D2" (shape input) (at 169.545 78.74 0) (fields_autoplaced)
+    (effects (font (size 1.27 1.27)) (justify left))
+    (property "Intersheetrefs" "${INTERSHEET_REFS}" (at 175.0097 78.74 0)
+      (effects (font (size 1.27 1.27)) (justify left) hide)
+    )
+  )
   (global_label "LED2(M)" (shape input) (at 29.845 38.1 90) (fields_autoplaced)
     (effects (font (size 1.27 1.27)) (justify left))
@@
     )
   )
+  (global_label "D3" (shape input) (at 113.665 104.14 180) (fields_autoplaced)
+    (effects (font (size 1.27 1.27)) (justify right))
+    (property "Intersheetrefs" "${INTERSHEET_REFS}" (at 108.2003 104.14 0)
+      (effects (font (size 1.27 1.27)) (justify right) hide)
+    )
+  )
   (global_label "S2" (shape input) (at 169.545 71.12 0) (fields_autoplaced)
     (effects (font (size 1.27 1.27)) (justify left))
@@
     )
   )
+  (global_label "STROBE" (shape input) (at 113.665 101.6 180) (fields_autoplaced)
+    (effects (font (size 1.27 1.27)) (justify right))
+    (property "Intersheetrefs" "${INTERSHEET_REFS}" (at 103.4832 101.6 0)
+      (effects (font (size 1.27 1.27)) (justify right) hide)
+    )
+  )
   (global_label "CAN_TD(M)" (shape input) (at 169.545 83.82 0) (fields_autoplaced)
     (effects (font (size 1.27 1.27)) (justify left))
@@
     )
   )
+  (global_label "BUSY" (shape input) (at 113.665 99.06 180) (fields_autoplaced)
+    (effects (font (size 1.27 1.27)) (justify right))
+    (property "Intersheetrefs" "${INTERSHEET_REFS}" (at 105.7812 99.06 0)
+      (effects (font (size 1.27 1.27)) (justify right) hide)
+    )
+  )
   (global_label "LED1(M)" (shape input) (at 20.32 38.1 90) (fields_autoplaced)
     (effects (font (size 1.27 1.27)) (justify left))
@@
       (effects (font (size 1.27 1.27)) (justify left) hide)
     )
+  )
+  (global_label "D1" (shape input) (at 169.545 109.22 0) (fields_autoplaced)
+    (effects (font (size 1.27 1.27)) (justify left))
+    (property "Intersheetrefs" "${INTERSHEET_REFS}" (at 175.0097 109.22 0)
+      (effects (font (size 1.27 1.27)) (justify left) hide)
+    )

Commit message: update
Connections:
- net +3.3V: no longer names the net of U4.16 (+3V3)
- no-connect marks 34 -> 35
Changed lines of the file:
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@@
   (no_connect (at 131.445 40.64))
   (no_connect (at 169.545 101.6))
+  (no_connect (at 133.985 40.64))
   (no_connect (at 169.545 58.42))
   (no_connect (at 113.665 119.38))
@@
     (stroke (width 0) (type default))
   )
-  (wire (pts (xy 133.985 39.37) (xy 132.08 39.37))
-    (stroke (width 0) (type default))
-  )
   (wire (pts (xy 20.955 82.55) (xy 20.955 84.455))
     (stroke (width 0) (type default))
@@
     (stroke (width 0) (type default))
   )
-  (wire (pts (xy 133.985 40.64) (xy 133.985 39.37))
-    (stroke (width 0) (type default))
-  )
   (wire (pts (xy 39.37 49.53) (xy 48.895 49.53))
     (stroke (width 0) (type default))
@@
   )
   (wire (pts (xy 136.525 39.37) (xy 138.43 39.37))
-    (stroke (width 0) (type default))
-  )
-  (wire (pts (xy 132.08 39.37) (xy 132.08 38.1))
     (stroke (width 0) (type default))
   )
@@
         )
       )
-    )
-  )
-  (symbol (lib_id "power:+3.3V") (at 132.08 38.1 0) (unit 1)
-    (in_bom yes) (on_board yes) (dnp no) (fields_autoplaced)
-    (property "Reference" "#PWR03" (at 132.08 41.91 0)
-      (effects (font (size 1.27 1.27)) hide)
-    )
-    (property "Value" "+3.3V" (at 132.08 33.9669 0)
-      (effects (font (size 1.27 1.27)))
-    )
-    (property "Footprint" "" (at 132.08 38.1 0)
-      (effects (font (size 1.27 1.27)) hide)
-    )
-    (property "Datasheet" "" (at 132.08 38.1 0)
-      (effects (font (size 1.27 1.27)) hide)
-    )
-    (pin "1")
-    (instances
-      (project "TVZ_KTM_ApplicationBoard"
-        (path "/e6e1ba2c-0a46-4bca-b3ad-33e778ea698b/7b36bbe9-69d8-437c-a840-f4b4d6c93da6"
-          (reference "#PWR03") (unit 1)
-        )
-      )

Commit message: update
Connections:
- net LED3(M): now also U4.36 (PC1); no longer U4.21 (PB7)
- net LED4(M): now also U4.38 (PC0); no longer U4.17 (PA15)
- net LED5(M): now also U4.17 (PA15); no longer U4.32 (PA4)
- net LED6(M): now also U4.51 (PA6); no longer U4.34 (PB0)
- net LED7(M): now also U4.53 (PA7); no longer U4.36 (PC1)
- net LED8(M): now also U4.61 (PA8); no longer U4.38 (PC0)
- net S1: now also U4.3 (PC12); no longer U4.57 (PC7)
- net S2: now also U4.1 (PC10); no longer U4.53 (PA7)
- net S3: now also U4.2 (PC11); no longer U4.55 (PB6)
- net S4: now also U4.57 (PC7); no longer U4.51 (PA6)
Changed lines of the file:
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@@
   (junction (at 37.465 95.885) (diameter 0) (color 0 0 0 0)
   )
-  (no_connect (at 169.545 73.66))
+  (no_connect (at 169.545 111.76))
   (no_connect (at 169.545 106.68))
   (no_connect (at 57.785 136.525))
@@
   (no_connect (at 169.545 104.14))
   (no_connect (at 139.065 40.64))
+  (no_connect (at 169.545 114.3))
   (no_connect (at 58.42 125.73))
   (no_connect (at 169.545 60.96))
   (no_connect (at 154.305 40.64))
-  (no_connect (at 113.665 124.46))
   (no_connect (at 144.145 40.64))
   (no_connect (at 131.445 40.64))
@@
   (no_connect (at 133.985 40.64))
   (no_connect (at 169.545 58.42))
-  (no_connect (at 113.665 119.38))
-  (no_connect (at 113.665 121.92))
+  (no_connect (at 169.545 63.5))
   (no_connect (at 128.905 40.64))
   (no_connect (at 113.665 88.9))
   (no_connect (at 169.545 99.06))
+  (no_connect (at 169.545 96.52))
   (no_connect (at 113.665 132.08))
   (no_connect (at 169.545 76.2))
@@
     (effects (font (size 1.27 1.27)) (justify left bottom))
   )
-  (global_label "S3" (shape input) (at 169.545 111.76 0) (fields_autoplaced)
-    (effects (font (size 1.27 1.27)) (justify left))
-    (property "Intersheetrefs" "${INTERSHEET_REFS}" (at 174.9492 111.76 0)
-      (effects (font (size 1.27 1.27)) (justify left) hide)
+  (global_label "S3" (shape input) (at 113.665 121.92 180) (fields_autoplaced)
+    (effects (font (size 1.27 1.27)) (justify right))
+    (property "Intersheetrefs" "${INTERSHEET_REFS}" (at 108.2608 121.92 0)
+      (effects (font (size 1.27 1.27)) (justify right) hide)
     )
   )
@@
     )
   )
-  (global_label "LED5(M)" (shape input) (at 169.545 63.5 0) (fields_autoplaced)
-    (effects (font (size 1.27 1.27)) (justify left))
-    (property "Intersheetrefs" "${INTERSHEET_REFS}" (at 180.3316 63.5 0)
+  (global_label "LED5(M)" (shape input) (at 169.545 91.44 0) (fields_autoplaced)
+    (effects (font (size 1.27 1.27)) (justify left))
+    (property "Intersheetrefs" "${INTERSHEET_REFS}" (at 180.3316 91.44 0)
       (effects (font (size 1.27 1.27)) (justify left) hide)
     )
@@
     )
   )
-  (global_label "S2" (shape input) (at 169.545 71.12 0) (fields_autoplaced)
-    (effects (font (size 1.27 1.27)) (justify left))
-    (property "Intersheetrefs" "${INTERSHEET_REFS}" (at 174.9492 71.12 0)
-      (effects (font (size 1.27 1.27)) (justify left) hide)
-    )
-  )
-  (global_label "S4" (shape input) (at 169.545 68.58 0) (fields_autoplaced)
-    (effects (font (size 1.27 1.27)) (justify left))
-    (property "Intersheetrefs" "${INTERSHEET_REFS}" (at 174.9492 68.58 0)
-      (effects (font (size 1.27 1.27)) (justify left) hide)
+  (global_label "S2" (shape input) (at 113.665 119.38 180) (fields_autoplaced)
+    (effects (font (size 1.27 1.27)) (justify right))
+    (property "Intersheetrefs" "${INTERSHEET_REFS}" (at 108.2608 119.38 0)
+      (effects (font (size 1.27 1.27)) (justify right) hide)
+    )
+  )
+  (global_label "S4" (shape input) (at 113.665 111.76 180) (fields_autoplaced)
+    (effects (font (size 1.27 1.27)) (justify right))
+    (property "Intersheetrefs" "${INTERSHEET_REFS}" (at 108.2608 111.76 0)
+      (effects (font (size 1.27 1.27)) (justify right) hide)
     )
   )
@@
     )
   )
-  (global_label "LED3(M)" (shape input) (at 169.545 114.3 0) (fields_autoplaced)
-    (effects (font (size 1.27 1.27)) (justify left))
-    (property "Intersheetrefs" "${INTERSHEET_REFS}" (at 180.3316 114.3 0)
-      (effects (font (size 1.27 1.27)) (justify left) hide)
+  (global_label "LED3(M)" (shape input) (at 113.665 96.52 180) (fields_autoplaced)
+    (effects (font (size 1.27 1.27)) (justify right))
+    (property "Intersheetrefs" "${INTERSHEET_REFS}" (at 102.8784 96.52 0)
+      (effects (font (size 1.27 1.27)) (justify right) hide)
     )
   )
@@
     )
   )
-  (global_label "LED8(M)" (shape input) (at 113.665 93.98 180) (fields_autoplaced)
+  (global_label "LED8(M)" (shape input) (at 169.545 73.66 0) (fields_autoplaced)
+    (effects (font (size 1.27 1.27)) (justify left))
+    (property "Intersheetrefs" "${INTERSHEET_REFS}" (at 180.3316 73.66 0)
+      (effects (font (size 1.27 1.27)) (justify left) hide)
+    )
+  )
+  (global_label "LED6(M)" (shape input) (at 169.545 68.58 0) (fields_autoplaced)
+    (effects (font (size 1.27 1.27)) (justify left))
+    (property "Intersheetrefs" "${INTERSHEET_REFS}" (at 180.3316 68.58 0)
+      (effects (font (size 1.27 1.27)) (justify left) hide)
+    )
+  )
+  (global_label "DAC(M)>>ADC(S)" (shape input) (at 107.95 172.085 0) (fields_autoplaced)
+    (effects (font (size 1.27 1.27)) (justify left))
+    (property "Intersheetrefs" "${INTERSHEET_REFS}" (at 127.3849 172.085 0)
+      (effects (font (size 1.27 1.27)) (justify left) hide)
+    )
+  )
+  (global_label "S1" (shape input) (at 48.26 128.27 180) (fields_autoplaced)
+    (effects (font (size 1.27 1.27)) (justify right))
+    (property "Intersheetrefs" "${INTERSHEET_REFS}" (at 42.8558 128.27 0)
+      (effects (font (size 1.27 1.27)) (justify right) hide)
+    )
+  )
+  (global_label "LED5(M)" (shape input) (at 20.955 82.55 90) (fields_autoplaced)
+    (effects (font (size 1.27 1.27)) (justify left))
+    (property "Intersheetrefs" "${INTERSHEET_REFS}" (at 20.955 71.7634 90)
+      (effects (font (size 1.27 1.27)) (justify left) hide)
+    )
+  )
+  (global_label "BUSY" (shape input) (at 113.665 99.06 180) (fields_autoplaced)
+    (effects (font (size 1.27 1.27)) (justify right))
+    (property "Intersheetrefs" "${INTERSHEET_REFS}" (at 105.7812 99.06 0)
+      (effects (font (size 1.27 1.27)) (justify right) hide)
+    )
+  )
+  (global_label "LED1(M)" (shape input) (at 20.32 38.1 90) (fields_autoplaced)
+    (effects (font (size 1.27 1.27)) (justify left))
+    (property "Intersheetrefs" "${INTERSHEET_REFS}" (at 20.32 27.3134 90)
+      (effects (font (size 1.27 1.27)) (justify left) hide)
+    )
+  )
+  (global_label "LED4(M)" (shape input) (at 113.665 93.98 180) (fields_autoplaced)
     (effects (font (size 1.27 1.27)) (justify right))
     (property "Intersheetrefs" "${INTERSHEET_REFS}" (at 102.8784 93.98 0)
@@
     )
   )
-  (global_label "LED6(M)" (shape input) (at 169.545 96.52 0) (fields_autoplaced)
-    (effects (font (size 1.27 1.27)) (justify left))
-    (property "Intersheetrefs" "${INTERSHEET_REFS}" (at 180.3316 96.52 0)
-      (effects (font (size 1.27 1.27)) (justify left) hide)
-    )
-  )
-  (global_label "DAC(M)>>ADC(S)" (shape input) (at 107.95 172.085 0) (fields_autoplaced)
-    (effects (font (size 1.27 1.27)) (justify left))
-    (property "Intersheetrefs" "${INTERSHEET_REFS}" (at 127.3849 172.085 0)
-      (effects (font (size 1.27 1.27)) (justify left) hide)
-    )
-  )
-  (global_label "S1" (shape input) (at 48.26 128.27 180) (fields_autoplaced)
-    (effects (font (size 1.27 1.27)) (justify right))
-    (property "Intersheetrefs" "${INTERSHEET_REFS}" (at 42.8558 128.27 0)
-      (effects (font (size 1.27 1.27)) (justify right) hide)
-    )
-  )
-  (global_label "LED5(M)" (shape input) (at 20.955 82.55 90) (fields_autoplaced)
-    (effects (font (size 1.27 1.27)) (justify left))
-    (property "Intersheetrefs" "${INTERSHEET_REFS}" (at 20.955 71.7634 90)
-      (effects (font (size 1.27 1.27)) (justify left) hide)
-    )
-  )
-  (global_label "BUSY" (shape input) (at 113.665 99.06 180) (fields_autoplaced)
-    (effects (font (size 1.27 1.27)) (justify right))
-    (property "Intersheetrefs" "${INTERSHEET_REFS}" (at 105.7812 99.06 0)
-      (effects (font (size 1.27 1.27)) (justify right) hide)
-    )
-  )
-  (global_label "LED1(M)" (shape input) (at 20.32 38.1 90) (fields_autoplaced)
-    (effects (font (size 1.27 1.27)) (justify left))
-    (property "Intersheetrefs" "${INTERSHEET_REFS}" (at 20.32 27.3134 90)
-      (effects (font (size 1.27 1.27)) (justify left) hide)
-    )
-  )
-  (global_label "LED4(M)" (shape input) (at 169.545 91.44 0) (fields_autoplaced)
-    (effects (font (size 1.27 1.27)) (justify left))
-    (property "Intersheetrefs" "${INTERSHEET_REFS}" (at 180.3316 91.44 0)
-      (effects (font (size 1.27 1.27)) (justify left) hide)
-    )
-  )
   (global_label "S2" (shape input) (at 47.625 139.065 180) (fields_autoplaced)
     (effects (font (size 1.27 1.27)) (justify right))
@@
     )
   )
-  (global_label "LED7(M)" (shape input) (at 113.665 96.52 180) (fields_autoplaced)
-    (effects (font (size 1.27 1.27)) (justify right))
-    (property "Intersheetrefs" "${INTERSHEET_REFS}" (at 102.8784 96.52 0)
-      (effects (font (size 1.27 1.27)) (justify right) hide)
+  (global_label "LED7(M)" (shape input) (at 169.545 71.12 0) (fields_autoplaced)
+    (effects (font (size 1.27 1.27)) (justify left))
+    (property "Intersheetrefs" "${INTERSHEET_REFS}" (at 180.3316 71.12 0)
+      (effects (font (size 1.27 1.27)) (justify left) hide)
     )
   )
@@
     )
   )
-  (global_label "S1" (shape input) (at 113.665 111.76 180) (fields_autoplaced)
-    (effects (font (size 1.27 1.27)) (justify right))
-    (property "Intersheetrefs" "${INTERSHEET_REFS}" (at 108.2608 111.76 0)
-      (effects (font (size 1.27 1.27)) (justify right) hide)
-    )
+  (global_label "S1" (shape input) (at 113.665 124.46 180) (fields_autoplaced)
+    (effects (font (size 1.27 1.27)) (justify right))
+    (property "Intersheetrefs" "${INTERSHEET_REFS}" (at 108.2608 124.46 0)
+      (effects (font (size 1.27 1.27)) (justify right) hide)
+    )

Commit message: update
Parts:
- R10, R11, R12, R13, R14, R15, R16, R17: value 220 -> 750
Other:
- note removed: "na lijevu stranu idu crvene i zelene"
- note removed: "sklopke idu na lijevu stranu"
Changed lines of the file:
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@@
     (stroke (width 0) (type default))
-  )
-  (text "sklopke idu na lijevu stranu" (at 41.275 176.53 0)
-    (effects (font (size 1.27 1.27)) (justify left bottom))
   )
   (text "DAC MASTER" (at 106.045 175.895 0)
     (effects (font (size 1.27 1.27)) (justify left bottom))
   )
-  (text "na lijevu stranu idu crvene i zelene" (at 18.415 109.22 0)
-    (effects (font (size 1.27 1.27)) (justify left bottom))
-  )
   (global_label "S3" (shape input) (at 113.665 121.92 180) (fields_autoplaced)
     (effects (font (size 1.27 1.27)) (justify right))
@@
   (symbol (lib_id "Device:R_Small") (at 20.32 40.64 0) (unit 1)
     (in_bom yes) (on_board yes) (dnp no) (fields_autoplaced)
-    (property "Reference" "R14" (at 21.8186 39.8053 0)
-      (effects (font (size 1.27 1.27)) (justify left))
-    )
-    (property "Value" "220" (at 21.8186 42.3422 0)
+    (property "Reference" "R14" (at 21.8186 39.4279 0)
+      (effects (font (size 1.27 1.27)) (justify left))
+    )
+    (property "Value" "750" (at 21.8186 41.8521 0)
       (effects (font (size 1.27 1.27)) (justify left))
     )
@@
   (symbol (lib_id "Device:R_Small") (at 39.37 40.64 0) (unit 1)
     (in_bom yes) (on_board yes) (dnp no) (fields_autoplaced)
-    (property "Reference" "R16" (at 40.8686 39.8053 0)
-      (effects (font (size 1.27 1.27)) (justify left))
-    )
-    (property "Value" "220" (at 40.8686 42.3422 0)
+    (property "Reference" "R16" (at 40.8686 39.4279 0)
+      (effects (font (size 1.27 1.27)) (justify left))
+    )
+    (property "Value" "750" (at 40.8686 41.8521 0)
       (effects (font (size 1.27 1.27)) (justify left))
     )
@@
   (symbol (lib_id "Device:R_Small") (at 29.845 86.995 0) (unit 1)
     (in_bom yes) (on_board yes) (dnp no) (fields_autoplaced)
-    (property "Reference" "R11" (at 31.3436 86.1603 0)
-      (effects (font (size 1.27 1.27)) (justify left))
-    )
-    (property "Value" "220" (at 31.3436 88.6972 0)
+    (property "Reference" "R11" (at 31.3436 85.7829 0)
+      (effects (font (size 1.27 1.27)) (justify left))
+    )
+    (property "Value" "750" (at 31.3436 88.2071 0)
       (effects (font (size 1.27 1.27)) (justify left))
     )
@@
   (symbol (lib_id "Device:R_Small") (at 49.53 86.995 0) (unit 1)
     (in_bom yes) (on_board yes) (dnp no) (fields_autoplaced)
-    (property "Reference" "R13" (at 51.0286 86.1603 0)
-      (effects (font (size 1.27 1.27)) (justify left))
-    )
-    (property "Value" "220" (at 51.0286 88.6972 0)
+    (property "Reference" "R13" (at 51.0286 85.7829 0)
+      (effects (font (size 1.27 1.27)) (justify left))
+    )
+    (property "Value" "750" (at 51.0286 88.2071 0)
       (effects (font (size 1.27 1.27)) (justify left))
     )
@@
   (symbol (lib_id "Device:R_Small") (at 29.845 40.64 0) (unit 1)
     (in_bom yes) (on_board yes) (dnp no) (fields_autoplaced)
-    (property "Reference" "R15" (at 31.3436 39.8053 0)
-      (effects (font (size 1.27 1.27)) (justify left))
-    )
-    (property "Value" "220" (at 31.3436 42.3422 0)
+    (property "Reference" "R15" (at 31.3436 39.4279 0)
+      (effects (font (size 1.27 1.27)) (justify left))
+    )
+    (property "Value" "750" (at 31.3436 41.8521 0)
       (effects (font (size 1.27 1.27)) (justify left))
     )
@@
   (symbol (lib_id "Device:R_Small") (at 20.955 86.995 0) (unit 1)
     (in_bom yes) (on_board yes) (dnp no) (fields_autoplaced)
-    (property "Reference" "R10" (at 22.4536 86.1603 0)
-      (effects (font (size 1.27 1.27)) (justify left))
-    )
-    (property "Value" "220" (at 22.4536 88.6972 0)
+    (property "Reference" "R10" (at 22.4536 85.7829 0)
+      (effects (font (size 1.27 1.27)) (justify left))
+    )
+    (property "Value" "750" (at 22.4536 88.2071 0)
       (effects (font (size 1.27 1.27)) (justify left))
     )
@@
   (symbol (lib_id "Device:R_Small") (at 48.895 40.64 0) (unit 1)
     (in_bom yes) (on_board yes) (dnp no) (fields_autoplaced)
-    (property "Reference" "R17" (at 50.3936 39.8053 0)
-      (effects (font (size 1.27 1.27)) (justify left))
-    )
-    (property "Value" "220" (at 50.3936 42.3422 0)
+    (property "Reference" "R17" (at 50.3936 39.4279 0)
+      (effects (font (size 1.27 1.27)) (justify left))
+    )
+    (property "Value" "750" (at 50.3936 41.8521 0)
       (effects (font (size 1.27 1.27)) (justify left))
     )
@@
   (symbol (lib_id "Device:R_Small") (at 39.37 86.995 0) (unit 1)
     (in_bom yes) (on_board yes) (dnp no) (fields_autoplaced)
-    (property "Reference" "R12" (at 40.8686 86.1603 0)
-      (effects (font (size 1.27 1.27)) (justify left))
-    )
-    (property "Value" "220" (at 40.8686 88.6972 0)
-      (effects (font (size 1.27 1.27)) (justify left))
-    )
+    (property "Reference" "R12" (at 40.8686 85.7829 0)
+      (effects (font (size 1.27 1.27)) (justify left))
+    )
+    (property "Value" "750" (at 40.8686 88.2071 0)
+      (effects (font (size 1.27 1.27)) (justify left))
+    )

Commit message: update
Connections:
- net LED1(M): now also U4.39 (PC9); no longer U4.25 (PC14)
Changed lines of the file:
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@@
   (no_connect (at 57.785 136.525))
   (no_connect (at 113.665 53.34))
-  (no_connect (at 113.665 116.84))
   (no_connect (at 113.665 106.68))
   (no_connect (at 57.785 158.75))
@@
   (no_connect (at 113.665 83.82))
   (no_connect (at 169.545 88.9))
+  (no_connect (at 113.665 129.54))
   (no_connect (at 57.785 147.32))
   (no_connect (at 113.665 55.88))
@@
     )
   )
-  (global_label "LED1(M)" (shape input) (at 113.665 129.54 180) (fields_autoplaced)
-    (effects (font (size 1.27 1.27)) (justify right))
-    (property "Intersheetrefs" "${INTERSHEET_REFS}" (at 102.8784 129.54 0)
-      (effects (font (size 1.27 1.27)) (justify right) hide)
-    )
+  (global_label "LED1(M)" (shape input) (at 113.665 116.84 180) (fields_autoplaced)
+    (effects (font (size 1.27 1.27)) (justify right))
+    (property "Intersheetrefs" "${INTERSHEET_REFS}" (at 102.8784 116.84 0)
+      (effects (font (size 1.27 1.27)) (justify right) hide)
+    )
