File: KiCAD files/Slave.kicad_sch (KiCad schematic)
At the start: 11 parts, among them U5 NUCLEO64-F446RE

Commit message: update
Connections:
- net STROBE: now reaches U5.30 (PA1)
- net BUSY: now reaches U5.32 (PA4)
- net D4: now reaches U5.34 (PB0)
- net D3: now reaches U5.35 (PC2)
- net D2: now reaches U5.36 (PC1)
- net D1: now reaches U5.37 (PC3)
- no-connect marks 46 -> 41
Changed lines of the file:
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@@
   (no_connect (at 142.24 43.18))
   (no_connect (at 157.48 43.18))
-  (no_connect (at 172.72 58.42))
   (no_connect (at 172.72 73.66))
   (no_connect (at 172.72 55.88))
@@
   (no_connect (at 172.72 114.3))
   (no_connect (at 172.72 116.84))
-  (no_connect (at 116.84 104.14))
   (no_connect (at 116.84 116.84))
   (no_connect (at 116.84 55.88))
   (no_connect (at 116.84 119.38))
   (no_connect (at 116.84 129.54))
-  (no_connect (at 172.72 66.04))
+  (no_connect (at 66.675 70.485))
   (no_connect (at 172.72 101.6))
   (no_connect (at 116.84 91.44))
@@
   (no_connect (at 172.72 91.44))
   (no_connect (at 172.72 124.46))
-  (no_connect (at 116.84 99.06))
   (no_connect (at 172.72 60.96))
   (no_connect (at 116.84 114.3))
-  (no_connect (at 172.72 99.06))
-  (no_connect (at 116.84 101.6))
   (no_connect (at 139.7 43.18))
   (no_connect (at 172.72 109.22))
@@
     )
   )
+  (global_label "D2" (shape input) (at 116.84 99.06 180) (fields_autoplaced)
+    (effects (font (size 1.27 1.27)) (justify right))
+    (property "Intersheetrefs" "${INTERSHEET_REFS}" (at 111.3753 99.06 0)
+      (effects (font (size 1.27 1.27)) (justify right) hide)
+    )
+  )
   (global_label "USART_TX(M) >> USART_RX(S)" (shape input) (at 172.72 78.74 0) (fields_autoplaced)
     (effects (font (size 1.27 1.27)) (justify left))
@@
     )
   )
+  (global_label "D1" (shape input) (at 116.84 104.14 180) (fields_autoplaced)
+    (effects (font (size 1.27 1.27)) (justify right))
+    (property "Intersheetrefs" "${INTERSHEET_REFS}" (at 111.3753 104.14 0)
+      (effects (font (size 1.27 1.27)) (justify right) hide)
+    )
+  )
   (global_label "DAC(M)>>ADC(S)" (shape input) (at 116.84 96.52 180) (fields_autoplaced)
     (effects (font (size 1.27 1.27)) (justify right))
@@
     )
   )
+  (global_label "BUSY" (shape input) (at 172.72 66.04 0) (fields_autoplaced)
+    (effects (font (size 1.27 1.27)) (justify left))
+    (property "Intersheetrefs" "${INTERSHEET_REFS}" (at 180.6038 66.04 0)
+      (effects (font (size 1.27 1.27)) (justify left) hide)
+    )
+  )
+  (global_label "STROBE" (shape input) (at 172.72 58.42 0) (fields_autoplaced)
+    (effects (font (size 1.27 1.27)) (justify left))
+    (property "Intersheetrefs" "${INTERSHEET_REFS}" (at 182.9018 58.42 0)
+      (effects (font (size 1.27 1.27)) (justify left) hide)
+    )
+  )
   (global_label "LED2(S)" (shape input) (at 172.72 71.12 0) (fields_autoplaced)
     (effects (font (size 1.27 1.27)) (justify left))
@@
     )
   )
+  (global_label "D4" (shape input) (at 172.72 99.06 0) (fields_autoplaced)
+    (effects (font (size 1.27 1.27)) (justify left))
+    (property "Intersheetrefs" "${INTERSHEET_REFS}" (at 178.1847 99.06 0)
+      (effects (font (size 1.27 1.27)) (justify left) hide)
+    )
+  )
+  (global_label "D3" (shape input) (at 116.84 101.6 180) (fields_autoplaced)
+    (effects (font (size 1.27 1.27)) (justify right))
+    (property "Intersheetrefs" "${INTERSHEET_REFS}" (at 111.3753 101.6 0)
+      (effects (font (size 1.27 1.27)) (justify right) hide)
+    )
+  )

Commit message: update
Connections:
- net DAC(M)>>ADC(S): now also R20.1
- no-connect marks 41 -> 40
Changed lines of the file:
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@@
   (no_connect (at 116.84 119.38))
   (no_connect (at 116.84 129.54))
-  (no_connect (at 66.675 70.485))
   (no_connect (at 172.72 101.6))
   (no_connect (at 116.84 91.44))
@@
     )
   )
+  (global_label "DAC(M)>>ADC(S)" (shape input) (at 66.675 70.485 90) (fields_autoplaced)
+    (effects (font (size 1.27 1.27)) (justify left))
+    (property "Intersheetrefs" "${INTERSHEET_REFS}" (at 66.675 51.0501 90)
+      (effects (font (size 1.27 1.27)) (justify left) hide)
+    )
+  )

Commit message: update
Connections:
- net DAC(M)>>ADC(S): no longer R20.1
- net LED4(S): now also U5.44 (PC5); no longer U5.49 (PA5)
- net +3V3: now reaches U5.16 (+3V3)
- net VDD: now reaches U5.18 (+5V)
- new net DAC(S): R20.1, U5.49 (PA5)
- no-connect marks 40 -> 37
Changed lines of the file:
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@@
   (no_connect (at 172.72 55.88))
   (no_connect (at 116.84 134.62))
-  (no_connect (at 116.84 109.22))
   (no_connect (at 172.72 127))
   (no_connect (at 172.72 134.62))
@@
   (no_connect (at 172.72 60.96))
   (no_connect (at 116.84 114.3))
-  (no_connect (at 139.7 43.18))
   (no_connect (at 172.72 109.22))
   (no_connect (at 116.84 132.08))
   (no_connect (at 172.72 88.9))
   (no_connect (at 172.72 104.14))
-  (no_connect (at 137.16 43.18))
   (no_connect (at 147.32 43.18))
   (no_connect (at 172.72 76.2))
@@
     (stroke (width 0) (type default))
   )
+  (wire (pts (xy 139.7 41.91) (xy 139.7 43.18))
+    (stroke (width 0) (type default))
+  )
   (wire (pts (xy 30.48 70.485) (xy 30.48 71.755))
     (stroke (width 0) (type default))
@@
   )
   (wire (pts (xy 37.465 76.835) (xy 37.465 77.47))
+    (stroke (width 0) (type default))
+  )
+  (wire (pts (xy 137.16 37.465) (xy 137.16 43.18))
     (stroke (width 0) (type default))
   )
@@
     )
   )
-  (global_label "LED4(S)" (shape input) (at 172.72 68.58 0) (fields_autoplaced)
-    (effects (font (size 1.27 1.27)) (justify left))
-    (property "Intersheetrefs" "${INTERSHEET_REFS}" (at 183.2647 68.58 0)
-      (effects (font (size 1.27 1.27)) (justify left) hide)
+  (global_label "LED4(S)" (shape input) (at 116.84 109.22 180) (fields_autoplaced)
+    (effects (font (size 1.27 1.27)) (justify right))
+    (property "Intersheetrefs" "${INTERSHEET_REFS}" (at 106.2953 109.22 0)
+      (effects (font (size 1.27 1.27)) (justify right) hide)
     )
   )
@@
     (effects (font (size 1.27 1.27)) (justify left))
     (property "Intersheetrefs" "${INTERSHEET_REFS}" (at 45.085 59.9403 90)
+      (effects (font (size 1.27 1.27)) (justify left) hide)
+    )
+  )
+  (global_label "DAC(S)" (shape input) (at 172.72 68.58 0) (fields_autoplaced)
+    (effects (font (size 1.27 1.27)) (justify left))
+    (property "Intersheetrefs" "${INTERSHEET_REFS}" (at 182.2367 68.58 0)
       (effects (font (size 1.27 1.27)) (justify left) hide)
     )
@@
     )
   )
-  (global_label "DAC(M)>>ADC(S)" (shape input) (at 66.675 70.485 90) (fields_autoplaced)
-    (effects (font (size 1.27 1.27)) (justify left))
-    (property "Intersheetrefs" "${INTERSHEET_REFS}" (at 66.675 51.0501 90)
+  (global_label "DAC(S)" (shape input) (at 66.675 70.485 90) (fields_autoplaced)
+    (effects (font (size 1.27 1.27)) (justify left))
+    (property "Intersheetrefs" "${INTERSHEET_REFS}" (at 66.675 60.9683 90)
       (effects (font (size 1.27 1.27)) (justify left) hide)
     )
@@
         )
       )
+    )
+  )
+  (symbol (lib_id "power:+3V3") (at 137.16 37.465 0) (unit 1)
+    (in_bom yes) (on_board yes) (dnp no) (fields_autoplaced)
+    (property "Reference" "#PWR03" (at 137.16 41.275 0)
+      (effects (font (size 1.27 1.27)) hide)
+    )
+    (property "Value" "+3V3" (at 137.16 33.3319 0)
+      (effects (font (size 1.27 1.27)))
+    )
+    (property "Footprint" "" (at 137.16 37.465 0)
+      (effects (font (size 1.27 1.27)) hide)
+    )
+    (property "Datasheet" "" (at 137.16 37.465 0)
+      (effects (font (size 1.27 1.27)) hide)
+    )
+    (pin "1")
+    (instances
+      (project "TVZ_KTM_ApplicationBoard"
+        (path "/e6e1ba2c-0a46-4bca-b3ad-33e778ea698b/5131e22c-8c1d-4cfc-85c2-f588b7754c75"
+          (reference "#PWR03") (unit 1)
+        )
+      )
+    )
+  )
+  (symbol (lib_id "power:VDD") (at 139.7 41.91 0) (unit 1)
+    (in_bom yes) (on_board yes) (dnp no) (fields_autoplaced)
+    (property "Reference" "#PWR029" (at 139.7 45.72 0)
+      (effects (font (size 1.27 1.27)) hide)
+    )
+    (property "Value" "VDD" (at 139.7 37.7769 0)
+      (effects (font (size 1.27 1.27)))
+    )
+    (property "Footprint" "" (at 139.7 41.91 0)
+      (effects (font (size 1.27 1.27)) hide)
+    )
+    (property "Datasheet" "" (at 139.7 41.91 0)
+      (effects (font (size 1.27 1.27)) hide)
+    )
+    (pin "1")
+    (instances
+      (project "TVZ_KTM_ApplicationBoard"
+        (path "/e6e1ba2c-0a46-4bca-b3ad-33e778ea698b/5131e22c-8c1d-4cfc-85c2-f588b7754c75"
+          (reference "#PWR029") (unit 1)
+        )
+      )

Commit message: update
Connections:
- net LED1(S): now also U5.53 (PA7); no longer U5.52 (PA11)
- net LED2(S): now also U5.52 (PA11); no longer U5.51 (PA6)
- net LED3(S): now also U5.51 (PA6); no longer U5.50 (PA12)
- net LED4(S): now also U5.50 (PA12); no longer U5.44 (PC5)
Changed lines of the file:
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@@
   (no_connect (at 142.24 43.18))
   (no_connect (at 157.48 43.18))
-  (no_connect (at 172.72 73.66))
+  (no_connect (at 116.84 109.22))
   (no_connect (at 172.72 55.88))
   (no_connect (at 116.84 134.62))
@@
     )
   )
-  (global_label "LED4(S)" (shape input) (at 116.84 109.22 180) (fields_autoplaced)
-    (effects (font (size 1.27 1.27)) (justify right))
-    (property "Intersheetrefs" "${INTERSHEET_REFS}" (at 106.2953 109.22 0)
-      (effects (font (size 1.27 1.27)) (justify right) hide)
+  (global_label "LED4(S)" (shape input) (at 172.72 86.36 0) (fields_autoplaced)
+    (effects (font (size 1.27 1.27)) (justify left))
+    (property "Intersheetrefs" "${INTERSHEET_REFS}" (at 183.2647 86.36 0)
+      (effects (font (size 1.27 1.27)) (justify left) hide)
     )
   )
@@
     )
   )
-  (global_label "LED3(S)" (shape input) (at 172.72 86.36 0) (fields_autoplaced)
-    (effects (font (size 1.27 1.27)) (justify left))
-    (property "Intersheetrefs" "${INTERSHEET_REFS}" (at 183.2647 86.36 0)
+  (global_label "LED3(S)" (shape input) (at 172.72 71.12 0) (fields_autoplaced)
+    (effects (font (size 1.27 1.27)) (justify left))
+    (property "Intersheetrefs" "${INTERSHEET_REFS}" (at 183.2647 71.12 0)
       (effects (font (size 1.27 1.27)) (justify left) hide)
     )
@@
     )
   )
-  (global_label "LED2(S)" (shape input) (at 172.72 71.12 0) (fields_autoplaced)
-    (effects (font (size 1.27 1.27)) (justify left))
-    (property "Intersheetrefs" "${INTERSHEET_REFS}" (at 183.2647 71.12 0)
+  (global_label "LED2(S)" (shape input) (at 172.72 83.82 0) (fields_autoplaced)
+    (effects (font (size 1.27 1.27)) (justify left))
+    (property "Intersheetrefs" "${INTERSHEET_REFS}" (at 183.2647 83.82 0)
       (effects (font (size 1.27 1.27)) (justify left) hide)
     )
@@
     )
   )
-  (global_label "LED1(S)" (shape input) (at 172.72 83.82 0) (fields_autoplaced)
-    (effects (font (size 1.27 1.27)) (justify left))
-    (property "Intersheetrefs" "${INTERSHEET_REFS}" (at 183.2647 83.82 0)
-      (effects (font (size 1.27 1.27)) (justify left) hide)
-    )
+  (global_label "LED1(S)" (shape input) (at 172.72 73.66 0) (fields_autoplaced)
+    (effects (font (size 1.27 1.27)) (justify left))
+    (property "Intersheetrefs" "${INTERSHEET_REFS}" (at 183.2647 73.66 0)
+      (effects (font (size 1.27 1.27)) (justify left) hide)
+    )

Commit message: update
Parts:
- D13: value boja -> BLUE
- R20, R6, R7, R8, R9: value 220 -> 300
Other:
- note removed: "na desnu stranu plave"
Changed lines of the file:
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@@
     (stroke (width 0) (type default))
   )
-  (text "na desnu stranu plave" (at 56.515 88.9 0)
-    (effects (font (size 1.27 1.27)) (justify left bottom))
-  )
   (global_label "SPI_MOSI" (shape input) (at 116.84 127 180) (fields_autoplaced)
     (effects (font (size 1.27 1.27)) (justify right))
@@
   (symbol (lib_id "Device:R_Small") (at 45.085 74.295 0) (unit 1)
     (in_bom yes) (on_board yes) (dnp no) (fields_autoplaced)
-    (property "Reference" "R8" (at 46.5836 73.4603 0)
-      (effects (font (size 1.27 1.27)) (justify left))
-    )
-    (property "Value" "220" (at 46.5836 75.9972 0)
+    (property "Reference" "R8" (at 46.5836 73.0829 0)
+      (effects (font (size 1.27 1.27)) (justify left))
+    )
+    (property "Value" "300" (at 46.5836 75.5071 0)
       (effects (font (size 1.27 1.27)) (justify left))
     )
@@
   (symbol (lib_id "Device:R_Small") (at 37.465 74.295 0) (unit 1)
     (in_bom yes) (on_board yes) (dnp no) (fields_autoplaced)
-    (property "Reference" "R7" (at 38.9636 73.4603 0)
-      (effects (font (size 1.27 1.27)) (justify left))
-    )
-    (property "Value" "220" (at 38.9636 75.9972 0)
+    (property "Reference" "R7" (at 38.9636 73.0829 0)
+      (effects (font (size 1.27 1.27)) (justify left))
+    )
+    (property "Value" "300" (at 38.9636 75.5071 0)
       (effects (font (size 1.27 1.27)) (justify left))
     )
@@
   (symbol (lib_id "Device:R_Small") (at 30.48 74.295 0) (unit 1)
     (in_bom yes) (on_board yes) (dnp no) (fields_autoplaced)
-    (property "Reference" "R6" (at 31.9786 73.4603 0)
-      (effects (font (size 1.27 1.27)) (justify left))
-    )
-    (property "Value" "220" (at 31.9786 75.9972 0)
+    (property "Reference" "R6" (at 31.9786 73.0829 0)
+      (effects (font (size 1.27 1.27)) (justify left))
+    )
+    (property "Value" "300" (at 31.9786 75.5071 0)
       (effects (font (size 1.27 1.27)) (justify left))
     )
@@
       (effects (font (size 1.27 1.27)) (justify right))
     )
-    (property "Value" "boja" (at 67.945 81.915 90)
+    (property "Value" "BLUE" (at 67.945 81.915 90)
       (effects (font (size 1.27 1.27)) (justify right))
     )
@@
   (symbol (lib_id "Device:R_Small") (at 66.675 74.295 0) (unit 1)
     (in_bom yes) (on_board yes) (dnp no) (fields_autoplaced)
-    (property "Reference" "R20" (at 68.1736 73.4603 0)
-      (effects (font (size 1.27 1.27)) (justify left))
-    )
-    (property "Value" "220" (at 68.1736 75.9972 0)
+    (property "Reference" "R20" (at 68.1736 73.0829 0)
+      (effects (font (size 1.27 1.27)) (justify left))
+    )
+    (property "Value" "300" (at 68.1736 75.5071 0)
       (effects (font (size 1.27 1.27)) (justify left))
     )
@@
   (symbol (lib_id "Device:R_Small") (at 52.705 74.295 0) (unit 1)
     (in_bom yes) (on_board yes) (dnp no) (fields_autoplaced)
-    (property "Reference" "R9" (at 54.2036 73.4603 0)
-      (effects (font (size 1.27 1.27)) (justify left))
-    )
-    (property "Value" "220" (at 54.2036 75.9972 0)
-      (effects (font (size 1.27 1.27)) (justify left))
-    )
+    (property "Reference" "R9" (at 54.2036 73.0829 0)
+      (effects (font (size 1.27 1.27)) (justify left))
+    )
+    (property "Value" "300" (at 54.2036 75.5071 0)
+      (effects (font (size 1.27 1.27)) (justify left))
+    )

Commit message: update
Connections:
- net LED1(S): now also U5.51 (PA6); no longer U5.53 (PA7)
- net LED2(S): now also U5.53 (PA7); no longer U5.52 (PA11)
- net LED3(S): now also U5.52 (PA11); no longer U5.51 (PA6)
Changed lines of the file:
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@@
     )
   )
-  (global_label "LED3(S)" (shape input) (at 172.72 71.12 0) (fields_autoplaced)
+  (global_label "LED3(S)" (shape input) (at 172.72 83.82 0) (fields_autoplaced)
     (effects (font (size 1.27 1.27)) (justify left))
-    (property "Intersheetrefs" "${INTERSHEET_REFS}" (at 183.2647 71.12 0)
+    (property "Intersheetrefs" "${INTERSHEET_REFS}" (at 183.2647 83.82 0)
       (effects (font (size 1.27 1.27)) (justify left) hide)
     )
@@
     )
   )
-  (global_label "LED2(S)" (shape input) (at 172.72 83.82 0) (fields_autoplaced)
+  (global_label "LED2(S)" (shape input) (at 172.72 73.66 0) (fields_autoplaced)
     (effects (font (size 1.27 1.27)) (justify left))
-    (property "Intersheetrefs" "${INTERSHEET_REFS}" (at 183.2647 83.82 0)
+    (property "Intersheetrefs" "${INTERSHEET_REFS}" (at 183.2647 73.66 0)
       (effects (font (size 1.27 1.27)) (justify left) hide)
     )
@@
     )
   )
-  (global_label "LED1(S)" (shape input) (at 172.72 73.66 0) (fields_autoplaced)
+  (global_label "LED1(S)" (shape input) (at 172.72 71.12 0) (fields_autoplaced)
     (effects (font (size 1.27 1.27)) (justify left))
-    (property "Intersheetrefs" "${INTERSHEET_REFS}" (at 183.2647 73.66 0)
+    (property "Intersheetrefs" "${INTERSHEET_REFS}" (at 183.2647 71.12 0)
       (effects (font (size 1.27 1.27)) (justify left) hide)
     )

Commit message: update
Connections:
- net D1: now also U5.38 (PC0); no longer U5.37 (PC3)
- net D4: now also U5.37 (PC3); no longer U5.34 (PB0)
- net DAC(M)>>ADC(S): now also U5.34 (PB0); no longer U5.38 (PC0)
Changed lines of the file:
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@@
   (no_connect (at 172.72 101.6))
   (no_connect (at 116.84 91.44))
-  (no_connect (at 116.84 106.68))
   (no_connect (at 172.72 106.68))
   (no_connect (at 172.72 91.44))
@@
   (no_connect (at 172.72 88.9))
   (no_connect (at 172.72 104.14))
+  (no_connect (at 116.84 106.68))
   (no_connect (at 147.32 43.18))
   (no_connect (at 172.72 76.2))
@@
     )
   )
-  (global_label "D1" (shape input) (at 116.84 104.14 180) (fields_autoplaced)
+  (global_label "D1" (shape input) (at 116.84 96.52 180) (fields_autoplaced)
+    (effects (font (size 1.27 1.27)) (justify right))
+    (property "Intersheetrefs" "${INTERSHEET_REFS}" (at 111.3753 96.52 0)
+      (effects (font (size 1.27 1.27)) (justify right) hide)
+    )
+  )
+  (global_label "DAC(M)>>ADC(S)" (shape input) (at 172.72 99.06 0) (fields_autoplaced)
+    (effects (font (size 1.27 1.27)) (justify left))
+    (property "Intersheetrefs" "${INTERSHEET_REFS}" (at 192.1549 99.06 0)
+      (effects (font (size 1.27 1.27)) (justify left) hide)
+    )
+  )
+  (global_label "LED4(S)" (shape input) (at 172.72 86.36 0) (fields_autoplaced)
+    (effects (font (size 1.27 1.27)) (justify left))
+    (property "Intersheetrefs" "${INTERSHEET_REFS}" (at 183.2647 86.36 0)
+      (effects (font (size 1.27 1.27)) (justify left) hide)
+    )
+  )
+  (global_label "CAN_RD(S)" (shape input) (at 172.72 111.76 0) (fields_autoplaced)
+    (effects (font (size 1.27 1.27)) (justify left))
+    (property "Intersheetrefs" "${INTERSHEET_REFS}" (at 185.8048 111.76 0)
+      (effects (font (size 1.27 1.27)) (justify left) hide)
+    )
+  )
+  (global_label "LED3(S)" (shape input) (at 172.72 83.82 0) (fields_autoplaced)
+    (effects (font (size 1.27 1.27)) (justify left))
+    (property "Intersheetrefs" "${INTERSHEET_REFS}" (at 183.2647 83.82 0)
+      (effects (font (size 1.27 1.27)) (justify left) hide)
+    )
+  )
+  (global_label "BUSY" (shape input) (at 172.72 66.04 0) (fields_autoplaced)
+    (effects (font (size 1.27 1.27)) (justify left))
+    (property "Intersheetrefs" "${INTERSHEET_REFS}" (at 180.6038 66.04 0)
+      (effects (font (size 1.27 1.27)) (justify left) hide)
+    )
+  )
+  (global_label "STROBE" (shape input) (at 172.72 58.42 0) (fields_autoplaced)
+    (effects (font (size 1.27 1.27)) (justify left))
+    (property "Intersheetrefs" "${INTERSHEET_REFS}" (at 182.9018 58.42 0)
+      (effects (font (size 1.27 1.27)) (justify left) hide)
+    )
+  )
+  (global_label "LED2(S)" (shape input) (at 172.72 73.66 0) (fields_autoplaced)
+    (effects (font (size 1.27 1.27)) (justify left))
+    (property "Intersheetrefs" "${INTERSHEET_REFS}" (at 183.2647 73.66 0)
+      (effects (font (size 1.27 1.27)) (justify left) hide)
+    )
+  )
+  (global_label "USART_RX(M) >> USART_TX(S)" (shape input) (at 172.72 81.28 0) (fields_autoplaced)
+    (effects (font (size 1.27 1.27)) (justify left))
+    (property "Intersheetrefs" "${INTERSHEET_REFS}" (at 205.1571 81.28 0)
+      (effects (font (size 1.27 1.27)) (justify left) hide)
+    )
+  )
+  (global_label "LED3(S)" (shape input) (at 45.085 70.485 90) (fields_autoplaced)
+    (effects (font (size 1.27 1.27)) (justify left))
+    (property "Intersheetrefs" "${INTERSHEET_REFS}" (at 45.085 59.9403 90)
+      (effects (font (size 1.27 1.27)) (justify left) hide)
+    )
+  )
+  (global_label "DAC(S)" (shape input) (at 172.72 68.58 0) (fields_autoplaced)
+    (effects (font (size 1.27 1.27)) (justify left))
+    (property "Intersheetrefs" "${INTERSHEET_REFS}" (at 182.2367 68.58 0)
+      (effects (font (size 1.27 1.27)) (justify left) hide)
+    )
+  )
+  (global_label "D4" (shape input) (at 116.84 104.14 180) (fields_autoplaced)
     (effects (font (size 1.27 1.27)) (justify right))
     (property "Intersheetrefs" "${INTERSHEET_REFS}" (at 111.3753 104.14 0)
@@
     )
   )
-  (global_label "DAC(M)>>ADC(S)" (shape input) (at 116.84 96.52 180) (fields_autoplaced)
-    (effects (font (size 1.27 1.27)) (justify right))
-    (property "Intersheetrefs" "${INTERSHEET_REFS}" (at 97.4051 96.52 0)
-      (effects (font (size 1.27 1.27)) (justify right) hide)
-    )
-  )
-  (global_label "LED4(S)" (shape input) (at 172.72 86.36 0) (fields_autoplaced)
-    (effects (font (size 1.27 1.27)) (justify left))
-    (property "Intersheetrefs" "${INTERSHEET_REFS}" (at 183.2647 86.36 0)
-      (effects (font (size 1.27 1.27)) (justify left) hide)
-    )
-  )
-  (global_label "CAN_RD(S)" (shape input) (at 172.72 111.76 0) (fields_autoplaced)
-    (effects (font (size 1.27 1.27)) (justify left))
-    (property "Intersheetrefs" "${INTERSHEET_REFS}" (at 185.8048 111.76 0)
-      (effects (font (size 1.27 1.27)) (justify left) hide)
-    )
-  )
-  (global_label "LED3(S)" (shape input) (at 172.72 83.82 0) (fields_autoplaced)
-    (effects (font (size 1.27 1.27)) (justify left))
-    (property "Intersheetrefs" "${INTERSHEET_REFS}" (at 183.2647 83.82 0)
-      (effects (font (size 1.27 1.27)) (justify left) hide)
-    )
-  )
-  (global_label "BUSY" (shape input) (at 172.72 66.04 0) (fields_autoplaced)
-    (effects (font (size 1.27 1.27)) (justify left))
-    (property "Intersheetrefs" "${INTERSHEET_REFS}" (at 180.6038 66.04 0)
-      (effects (font (size 1.27 1.27)) (justify left) hide)
-    )
-  )
-  (global_label "STROBE" (shape input) (at 172.72 58.42 0) (fields_autoplaced)
-    (effects (font (size 1.27 1.27)) (justify left))
-    (property "Intersheetrefs" "${INTERSHEET_REFS}" (at 182.9018 58.42 0)
-      (effects (font (size 1.27 1.27)) (justify left) hide)
-    )
-  )
-  (global_label "LED2(S)" (shape input) (at 172.72 73.66 0) (fields_autoplaced)
-    (effects (font (size 1.27 1.27)) (justify left))
-    (property "Intersheetrefs" "${INTERSHEET_REFS}" (at 183.2647 73.66 0)
-      (effects (font (size 1.27 1.27)) (justify left) hide)
-    )
-  )
-  (global_label "USART_RX(M) >> USART_TX(S)" (shape input) (at 172.72 81.28 0) (fields_autoplaced)
-    (effects (font (size 1.27 1.27)) (justify left))
-    (property "Intersheetrefs" "${INTERSHEET_REFS}" (at 205.1571 81.28 0)
-      (effects (font (size 1.27 1.27)) (justify left) hide)
-    )
-  )
-  (global_label "LED3(S)" (shape input) (at 45.085 70.485 90) (fields_autoplaced)
-    (effects (font (size 1.27 1.27)) (justify left))
-    (property "Intersheetrefs" "${INTERSHEET_REFS}" (at 45.085 59.9403 90)
-      (effects (font (size 1.27 1.27)) (justify left) hide)
-    )
-  )
-  (global_label "DAC(S)" (shape input) (at 172.72 68.58 0) (fields_autoplaced)
-    (effects (font (size 1.27 1.27)) (justify left))
-    (property "Intersheetrefs" "${INTERSHEET_REFS}" (at 182.2367 68.58 0)
-      (effects (font (size 1.27 1.27)) (justify left) hide)
-    )
-  )
-  (global_label "D4" (shape input) (at 172.72 99.06 0) (fields_autoplaced)
-    (effects (font (size 1.27 1.27)) (justify left))
-    (property "Intersheetrefs" "${INTERSHEET_REFS}" (at 178.1847 99.06 0)
-      (effects (font (size 1.27 1.27)) (justify left) hide)
-    )
-  )
