File: KiCAD files/Slave.kicad_sch (KiCad schematic)
At the start: 11 parts, among them U5 NUCLEO64-F446RE

Commit message: update
Connections:
- net D4 is gone; now on net D3: U5.37 (PC3)
- net D2: now also U5.35 (PC2); no longer U5.36 (PC1)
- net D3: no longer U5.35 (PC2)
- net LED1(S): now also U5.50 (PA12); no longer U5.51 (PA6)
- net LED2(S): now also U5.52 (PA11); no longer U5.53 (PA7)
- net LED3(S): now also U5.53 (PA7); no longer U5.52 (PA11)
- net LED4(S): now also U5.51 (PA6); no longer U5.50 (PA12)
- new net D0: U5.36 (PC1)
Changed lines of the file:
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@@
     )
   )
-  (global_label "D2" (shape input) (at 116.84 99.06 180) (fields_autoplaced)
+  (global_label "D1" (shape input) (at 116.84 96.52 180) (fields_autoplaced)
     (effects (font (size 1.27 1.27)) (justify right))
-    (property "Intersheetrefs" "${INTERSHEET_REFS}" (at 111.3753 99.06 0)
+    (property "Intersheetrefs" "${INTERSHEET_REFS}" (at 111.3753 96.52 0)
       (effects (font (size 1.27 1.27)) (justify right) hide)
     )
@@
     )
   )
-  (global_label "D1" (shape input) (at 116.84 96.52 180) (fields_autoplaced)
+  (global_label "D0" (shape input) (at 116.84 99.06 180) (fields_autoplaced)
     (effects (font (size 1.27 1.27)) (justify right))
-    (property "Intersheetrefs" "${INTERSHEET_REFS}" (at 111.3753 96.52 0)
+    (property "Intersheetrefs" "${INTERSHEET_REFS}" (at 111.3753 99.06 0)
       (effects (font (size 1.27 1.27)) (justify right) hide)
     )
@@
     )
   )
-  (global_label "LED4(S)" (shape input) (at 172.72 86.36 0) (fields_autoplaced)
+  (global_label "LED4(S)" (shape input) (at 172.72 71.12 0) (fields_autoplaced)
     (effects (font (size 1.27 1.27)) (justify left))
-    (property "Intersheetrefs" "${INTERSHEET_REFS}" (at 183.2647 86.36 0)
+    (property "Intersheetrefs" "${INTERSHEET_REFS}" (at 183.2647 71.12 0)
       (effects (font (size 1.27 1.27)) (justify left) hide)
     )
@@
     )
   )
-  (global_label "LED3(S)" (shape input) (at 172.72 83.82 0) (fields_autoplaced)
+  (global_label "LED3(S)" (shape input) (at 172.72 73.66 0) (fields_autoplaced)
     (effects (font (size 1.27 1.27)) (justify left))
-    (property "Intersheetrefs" "${INTERSHEET_REFS}" (at 183.2647 83.82 0)
+    (property "Intersheetrefs" "${INTERSHEET_REFS}" (at 183.2647 73.66 0)
       (effects (font (size 1.27 1.27)) (justify left) hide)
     )
@@
     )
   )
-  (global_label "LED2(S)" (shape input) (at 172.72 73.66 0) (fields_autoplaced)
+  (global_label "LED2(S)" (shape input) (at 172.72 83.82 0) (fields_autoplaced)
     (effects (font (size 1.27 1.27)) (justify left))
-    (property "Intersheetrefs" "${INTERSHEET_REFS}" (at 183.2647 73.66 0)
+    (property "Intersheetrefs" "${INTERSHEET_REFS}" (at 183.2647 83.82 0)
       (effects (font (size 1.27 1.27)) (justify left) hide)
     )
@@
     )
   )
-  (global_label "D4" (shape input) (at 116.84 104.14 180) (fields_autoplaced)
+  (global_label "D3" (shape input) (at 116.84 104.14 180) (fields_autoplaced)
     (effects (font (size 1.27 1.27)) (justify right))
     (property "Intersheetrefs" "${INTERSHEET_REFS}" (at 111.3753 104.14 0)
@@
     )
   )
-  (global_label "D3" (shape input) (at 116.84 101.6 180) (fields_autoplaced)
+  (global_label "D2" (shape input) (at 116.84 101.6 180) (fields_autoplaced)
     (effects (font (size 1.27 1.27)) (justify right))
     (property "Intersheetrefs" "${INTERSHEET_REFS}" (at 111.3753 101.6 0)
@@
     )
   )
-  (global_label "LED1(S)" (shape input) (at 172.72 71.12 0) (fields_autoplaced)
+  (global_label "LED1(S)" (shape input) (at 172.72 86.36 0) (fields_autoplaced)
     (effects (font (size 1.27 1.27)) (justify left))
-    (property "Intersheetrefs" "${INTERSHEET_REFS}" (at 183.2647 71.12 0)
+    (property "Intersheetrefs" "${INTERSHEET_REFS}" (at 183.2647 86.36 0)
       (effects (font (size 1.27 1.27)) (justify left) hide)
     )
