File: KiCAD files/Slave.kicad_sch (KiCad schematic)
At the start: 11 parts, among them U5 NUCLEO64-F446RE

Commit message: update
Connections:
- net USART_RX(M) >> USART_TX(S): now also U5.59 (PA9); no longer U5.71 (PA10)
- net USART_TX(M) >> USART_RX(S): now also U5.71 (PA10); no longer U5.59 (PA9)
Changed lines of the file:
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@@
     )
   )
-  (global_label "USART_TX(M) >> USART_RX(S)" (shape input) (at 172.72 78.74 0) (fields_autoplaced)
+  (global_label "USART_TX(M) >> USART_RX(S)" (shape input) (at 172.72 81.28 0) (fields_autoplaced)
     (effects (font (size 1.27 1.27)) (justify left))
-    (property "Intersheetrefs" "${INTERSHEET_REFS}" (at 205.1571 78.74 0)
+    (property "Intersheetrefs" "${INTERSHEET_REFS}" (at 205.1571 81.28 0)
       (effects (font (size 1.27 1.27)) (justify left) hide)
     )
@@
     )
   )
-  (global_label "USART_RX(M) >> USART_TX(S)" (shape input) (at 172.72 81.28 0) (fields_autoplaced)
+  (global_label "USART_RX(M) >> USART_TX(S)" (shape input) (at 172.72 78.74 0) (fields_autoplaced)
     (effects (font (size 1.27 1.27)) (justify left))
-    (property "Intersheetrefs" "${INTERSHEET_REFS}" (at 205.1571 81.28 0)
+    (property "Intersheetrefs" "${INTERSHEET_REFS}" (at 205.1571 78.74 0)
       (effects (font (size 1.27 1.27)) (justify left) hide)
     )

Commit message: v1rev3
Parts:
- removed D13: BLUE, LED_SMD:LED_1206_3216Metric, symbol Device:LED_Small
- removed R20: 300, Resistor_SMD:R_0805_2012Metric, symbol Device:R_Small
Changed lines of the file:
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@@
   (junction (at 45.085 83.185) (diameter 0) (color 0 0 0 0)
-  )
-  (junction (at 52.705 83.185) (diameter 0) (color 0 0 0 0)
   )
   (junction (at 135.89 146.685) (diameter 0) (color 0 0 0 0)
@@
   (no_connect (at 116.84 58.42))
   (no_connect (at 144.78 43.18))
-  (wire (pts (xy 66.675 83.185) (xy 66.675 82.55))
-    (stroke (width 0) (type default))
-  )
   (wire (pts (xy 139.7 144.78) (xy 139.7 146.685))
     (stroke (width 0) (type default))
@@
     (stroke (width 0) (type default))
   )
-  (wire (pts (xy 52.705 83.185) (xy 66.675 83.185))
-    (stroke (width 0) (type default))
-  )
   (wire (pts (xy 45.085 83.185) (xy 45.085 83.82))
     (stroke (width 0) (type default))
@@
     (stroke (width 0) (type default))
   )
-  (wire (pts (xy 66.675 70.485) (xy 66.675 71.755))
-    (stroke (width 0) (type default))
-  )
   (wire (pts (xy 135.89 146.685) (xy 135.89 147.955))
     (stroke (width 0) (type default))
@@
     (stroke (width 0) (type default))
   )
-  (wire (pts (xy 66.675 76.835) (xy 66.675 77.47))
-    (stroke (width 0) (type default))
-  )
   (wire (pts (xy 37.465 82.55) (xy 37.465 83.185))
     (stroke (width 0) (type default))
@@
     (property "Intersheetrefs" "${INTERSHEET_REFS}" (at 105.2067 124.46 0)
       (effects (font (size 1.27 1.27)) (justify right) hide)
-    )
-  )
-  (global_label "DAC(S)" (shape input) (at 66.675 70.485 90) (fields_autoplaced)
-    (effects (font (size 1.27 1.27)) (justify left))
-    (property "Intersheetrefs" "${INTERSHEET_REFS}" (at 66.675 60.9683 90)
-      (effects (font (size 1.27 1.27)) (justify left) hide)
     )
   )
@@
         )
       )
-    )
-  )
-  (symbol (lib_id "Device:LED_Small") (at 66.675 80.01 90) (unit 1)
-    (in_bom yes) (on_board yes) (dnp no)
-    (property "Reference" "D13" (at 68.453 79.1118 90)
-      (effects (font (size 1.27 1.27)) (justify right))
-    )
-    (property "Value" "BLUE" (at 67.945 81.915 90)
-      (effects (font (size 1.27 1.27)) (justify right))
-    )
-    (property "Footprint" "LED_SMD:LED_1206_3216Metric" (at 66.675 80.01 90)
-      (effects (font (size 1.27 1.27)) hide)
-    )
-    (property "Datasheet" "~" (at 66.675 80.01 90)
-      (effects (font (size 1.27 1.27)) hide)
-    )
-    (pin "1")
-    (pin "2")
-    (instances
-      (project "TVZ_KTM_ApplicationBoard"
-        (path "/e6e1ba2c-0a46-4bca-b3ad-33e778ea698b"
-          (reference "D13") (unit 1)
-        )
-        (path "/e6e1ba2c-0a46-4bca-b3ad-33e778ea698b/5131e22c-8c1d-4cfc-85c2-f588b7754c75"
-          (reference "D13") (unit 1)
-        )
-      )
-    )
-  )
-  (symbol (lib_id "Device:R_Small") (at 66.675 74.295 0) (unit 1)
-    (in_bom yes) (on_board yes) (dnp no) (fields_autoplaced)
-    (property "Reference" "R20" (at 68.1736 73.0829 0)
-      (effects (font (size 1.27 1.27)) (justify left))
-    )
-    (property "Value" "300" (at 68.1736 75.5071 0)
-      (effects (font (size 1.27 1.27)) (justify left))
-    )
-    (property "Footprint" "Resistor_SMD:R_0805_2012Metric" (at 66.675 74.295 0)
-      (effects (font (size 1.27 1.27)) hide)
-    )
-    (property "Datasheet" "~" (at 66.675 74.295 0)
-      (effects (font (size 1.27 1.27)) hide)
-    )
-    (pin "1")
-    (pin "2")
-    (instances
-      (project "TVZ_KTM_ApplicationBoard"
-        (path "/e6e1ba2c-0a46-4bca-b3ad-33e778ea698b"
-          (reference "R20") (unit 1)
-        )
-        (path "/e6e1ba2c-0a46-4bca-b3ad-33e778ea698b/5131e22c-8c1d-4cfc-85c2-f588b7754c75"
-          (reference "R20") (unit 1)
-        )
-      )
